File: Hardware/Kicad/Kicad.kicad_sch (KiCad schematic)
At the start: 9 parts, among them U1 LV25-P, U2 LV25-P, U3 LV25-P

Commit message: Miseajour1
Parts:
- added J1, J2, J3, J4: Conn_01x01, Connector:Banana_Cliff_FCR7350B_S16N-PC_Horizontal, symbol Connector_Generic:Conn_01x01
- added J5: DA15_Receptacle_MountingHoles, symbol Connector:DA15_Receptacle_MountingHoles
- added R10, R11, R12, R13, R14, R15, R7, R8, R9: R, symbol Device:R
- added U4, U5, U6: OP275, symbol Amplifier_Operational:OP275
Connections:
- net at R6.2, U3.4 (M): now also U6.3 (+)
- net at R1.2: now also J1.1 (Pin_1)
- net at U2.3 (HV-): now also U1.3 (HV-), U3.3 (HV-), J4.1 (Pin_1)
- net at R5.2, U2.4 (M): now also U5.3 (+)
- net at R3.2: now also J3.1 (Pin_1)
- net at R2.2: now also J2.1 (Pin_1)
- net at R4.2, U1.4 (M): now also U4.3 (+)
- new net: R14.2, R15.2, U6.5 (+)
- new net: R8.2, R9.2, U4.5 (+)
- new net: J5.1, U4.6 (-), U4.7
- new net: R7.2, R9.1, U4.1
- new net: R7.1, U4.2 (-)
- new net: J5.3, U6.6 (-), U6.7
- new net: R10.2, R11.1, U5.1
- new net: R10.1, U5.2 (-)
- new net: R11.2, R12.2, U5.5 (+)
- new net: R13.2, R14.1, U6.1
- new net: R13.1, U6.2 (-)
- new net: J5.2, U5.6 (-), U5.7
Other:
- moved on the sheet: R1, R2, R3, R4, R5, R6, U1, U2, U3

Commit message: miseajour
Parts:
- added R16, R17, R18, R19, R20, R21, R22, R23, R24, R25, R26, R27, R28, R29, R30, R31: R, symbol Device:R
- added U10, U11, U12, U13, U14, U15, U8, U9: OP275, symbol Amplifier_Operational:OP275
- added U7: LM2937xS, Package_TO_SOT_SMD:TO-263-3_TabPin2, symbol Regulator_Linear:LM2937xS
Connections:
- net at U4.6 (-), U4.7: no longer J5.1
- net at U6.6 (-), U6.7: no longer J5.3
- net at U5.6 (-), U5.7: no longer J5.2
- new net: R24.1, R26.2, U12.1
- new net: R24.2, R25.1, U12.2 (-)
- new net: R28.1, R30.2, U14.1
- new net: R28.2, R29.1, U14.2 (-)
- new net: R20.2, R21.1, U10.2 (-)
- new net: U15.1, U15.2 (-)
- new net: R30.1, R31.2, U15.3 (+)
- new net: R16.1, R19.2, U8.1
- new net: R16.2, R17.1, U8.2 (-)
- new net: R22.1, R23.2, U11.3 (+)
- new net: R20.1, R22.2, U10.1
- new net: R26.1, R27.2, U13.3 (+)
- new net: U9.1, U9.2 (-)
- new net: R18.2, R19.1, U9.3 (+)
- new net: U11.1, U11.2 (-)
- new net: U13.1, U13.2 (-)
Other:
- moved on the sheet: J5, R10, R11, R12, R13, R14, R15, R7, R8, R9, U4A, U4B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
