File: Hardware/Kicad_Carte_Acquisition/Kicad.kicad_sch (KiCad schematic)
At the start: 51 parts, among them J1 Conn_01x01, J2 Conn_01x01, J3 Conn_01x01, J4 Conn_01x01, J5 DA15_Receptacle_MountingHoles, U1 LV25-P, U10 OP275, U11 OP275, U12 OP275, U13 OP275, U14 OP275, U15 OP275, U2 LV25-P, U3 LV25-P, U4 OP275, U5 OP275, U6 OP275, U7 LM2937xS, U8 OP275, U9 OP275

Commit message: modif
Parts:
- removed U10, U11, U12, U13, U14, U15: OP275, symbol Amplifier_Operational:OP275
- added C1, C2: C, symbol Device:C
- added J2, J3, J6, J7: Conn_Coaxial, symbol Connector:Conn_Coaxial
- added TP1, TP10, TP2, TP3, TP4, TP5, TP6, TP7, TP8, TP9: TestPoint, symbol Connector:TestPoint
- added unit 3 of U4
- added unit 3 of U5
- added unit 3 of U6
- added unit 2 of U8
- added unit 2 of U9
- renumbered J1 to J1_Vphase1, J2 to J2_Vphase2, J3 to J3_Vphase3, J4 to J4_Neutre
Connections:
- net +3V3: now reaches R15.1
- net +3V3: now also R12.1, R18.1, R23.1, R27.1, R31.1, R8.1, U7.3 (VO), C2.1
- net at R6.2, U3.4 (M), U6.3 (+): now also TP3.1
- net Vph1: now reaches U4.6 (-), U4.7
- net Vph1: now also J5.1, TP4.1
- net at R20.2, R21.1: now also U9.2 (-)
- net GND: now reaches R21.2
- net GND: now also J5.0 (PAD), R17.2, R25.2, R29.2, U7.2 (GND), C1.2, C2.2, J2.2 (Ext), J3.2 (Ext), J6.2 (Ext), J7.2 (Ext)
- net at R4.2, U1.4 (M), U4.3 (+): now also TP1.1
- net at R22.1, R23.2: now also U9.5 (+)
- net at R20.1, R22.2: now also U9.1
- net Vph3: now reaches U6.6 (-), U6.7
- net Vph3: now also J5.3, TP6.1
- net at R5.2, U2.4 (M), U5.3 (+): now also TP2.1
- net at R18.2, R19.1: now also U8.5 (+); no longer U9.3 (+)
- net +15V: now reaches U7.1 (VI)
- net +15V: now also C1.1
- net at U8.3 (+): now also J2.1 (In)
- net Vcurrent_ph2: now reaches J5.10 (P10)
- net Vcurrent_ph2: now also TP8.1, U9.6 (-), U9.7
- net Vcurrent_ph3: now reaches J5.11 (P111)
- net Vcurrent_ph3: now also TP9.1
- net Vph2: now reaches J5.2
- net Vph2: now also U5.6 (-), U5.7, TP5.1
- net Vcurrent_neutre: now reaches J5.4
- net Vcurrent_neutre: now also TP10.1
- net Vcurrent_ph1: now reaches J5.9 (P9)
- net Vcurrent_ph1: now also TP7.1, U8.6 (-), U8.7
- new net: J6.1 (In), U9.3 (+)
Other:
- moved on the sheet: J1_Vphase1, J4_Neutre, R13, R14, R15, R20, R21, R22, R23, R28, R29, R30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

Commit message: modif
Parts:
- removed unit 3 of U6
- added C10, C11, C12, C13, C14, C3, C4, C5, C6, C7, C8, C9: C, symbol Device:C
- added U10, U11: OP275, symbol Amplifier_Operational:OP275
- added U12: TMP-15-215, symbol New_Library.kicad_Traco_sym:TMP-15-215
- added unit 3 of U8
- added unit 3 of U9
Connections:
- net +15V: now also J5.15 (P15), U1.5 (V+), U2.5 (V+), U3.5 (V+), U4.8 (V+), U5.8 (V+), C3.1, C4.1, C5.1, C6.1, C7.1, C8.1, U10.8 (V+), U11.8 (V+), U12.6 (Vout1), U8.8 (V+), U9.8 (V+)
- net GND: now also J5.8, C10.2, C11.2, C12.2, C13.2, C14.2, C3.2, C4.2, C5.2, C6.2, C7.2, C8.2, C9.2, U12.5 (Comm)
- net Vcurrent_neutre: now also U11.6 (-), U11.7
- net Vcurrent_ph3: now also U10.6 (-), U10.7
- net at R24.1, R26.2: now also U10.1
- net at R24.2, R25.1: now also U10.2 (-)
- net -15V: now reaches U5.4 (V-)
- net -15V: now also U4.4 (V-), C10.1, C11.1, C12.1, C13.1, C14.1, C9.1, U10.4 (V-), U11.4 (V-), U12.4 (Vout2), U8.4 (V-), U9.4 (V-)
- net at J3.1 (In): now also U10.3 (+)
- net at R4.1, U1.6 (V-), U2.6 (V-): no longer R5.1, R6.1, U3.6 (V-)
- net at R26.1, R27.2: now also U10.5 (+)
- net at R28.2, R29.1: now also U11.2 (-)
- net at R28.1, R30.2: now also U11.1
- net at J7.1 (In): now also U11.3 (+)
- net at R30.1, R31.2: now also U11.5 (+)
Other:
- moved on the sheet: C1, C2, J2, J3, J5, J6, J7, R10, R11, R12, R13, R14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

Commit message: modif
Parts:
- removed J2, J3, J6, J7: Conn_Coaxial, symbol Connector:Conn_Coaxial
- removed R16, R17, R18, R19, R20, R21, R22, R23, R24, R25, R26, R27, R28, R29, R30, R31: R, symbol Device:R
- removed TP10, TP7, TP8, TP9: TestPoint, symbol Connector:TestPoint
- removed unit 2 of U10
- removed unit 1 of U10
- removed unit 2 of U11
- removed unit 1 of U11
- removed unit 1 of U8
- removed unit 2 of U8
- removed unit 1 of U9
- removed unit 2 of U9
- added J5_Ph_230V1, J6_Neutre_230V1: Conn_01x01, Connector:Banana_Cliff_FCR7350B_S16N-PC_Horizontal, symbol Connector_Generic:Conn_01x01
- U12: footprint (none) -> Library.pretty_Traco_TMP15215:TMP-15-215E
- renumbered J4_Neutre to J4_Neutre1, J5 to P1
Connections:
- net +15V: now also U1.6 (V-), U2.6 (V-), U3.6 (V-)
- net GND: now also R4.1, R5.1, R6.1
- net at U12.1 (AC(N)): now also J6_Neutre_230V1.1 (Pin_1)
- net at U12.2 (AC(L)): now also J5_Ph_230V1.1 (Pin_1)
Other:
- added sheet Conditionnement_Capteur_1 (Conditionnement_capteur.kicad_sch)
- added sheet Conditionnement_Capteur_2 (Conditionnement_capteur.kicad_sch)
- added sheet Conditionnement_Capteur_3 (Conditionnement_capteur.kicad_sch)
- added sheet Conditionnement_Capteur_4 (Conditionnement_capteur.kicad_sch)
- moved on the sheet: R6

Commit message: modif
Parts:
- removed J2_Vphase2, J3_Vphase3, J4_Neutre1: Conn_01x01, Connector:Banana_Cliff_FCR7350B_S16N-PC_Horizontal, symbol Connector_Generic:Conn_01x01
- removed R10, R11, R12, R13, R14, R15, R3, R4, R5, R6, R7, R8, R9: R, symbol Device:R
- removed TP1, TP2, TP3, TP4, TP5, TP6: TestPoint, symbol Connector:TestPoint
- removed U1, U2, U3: LV25-P, Sensor_Voltage:LEM_LV25-P, symbol Sensor_Voltage:LV25-P
- removed unit 2 of U4
- removed unit 1 of U4
- removed unit 1 of U5
- removed unit 2 of U5
- removed U6: OP275, symbol Amplifier_Operational:OP275
- added D1, D2: LED_Small, symbol Device:LED_Small
- added J1_Vphase2, J1_Vphase3, J1_Vphase4: Conn_01x01, Connector:Banana_Cliff_FCR7350B_S16N-PC_Horizontal, symbol Connector_Generic:Conn_01x01
- C1, C2: value C -> 10uF
- C10, C11, C13, C14, C4, C9: value C -> 0.1uF
- C3: renamed from C8; value C -> 0.1uF
- C6: renamed from C3; value C -> 0.1uF
- C7: renamed from C6; value C -> 0.1uF
- C8: renamed from C7; value C -> 0.1uF
- R1, R2: value R -> 7.5k
- renumbered U12 to U1, U7 to U2, U4 to U3, U5 to U4, U8 to U5, U9 to U6, U10 to U7, U11 to U8
Connections:
- net +15V: now also R1.2
- net -15V: now also R2.1
- net GND: now also D1.1 (K), D2.2 (A)
- net at R1.1: now also D1.2 (A)
- net Cond_Capt_Tension_Ph1/J_Conn_in: now reaches J1_Vphase1.1 (Pin_1)
- net Cond_Capt_Tension_Ph1/J_Conn_in: no longer R1.2
- net at R2.2: now also D2.1 (K)
- new net Cond_Capt_Tension_Ph2/J_Conn_in: J1_Vphase3.1 (Pin_1)
- new net Cond_Capt_Tension_Ph3/J_Conn_in: J1_Vphase2.1 (Pin_1)
- new net Cond_Capt_Tension_Ph4/J_Conn_in: J1_Vphase4.1 (Pin_1)
Other:
- added sheet Cond_Capt_Tension_Ph1 (Cond_Capt_Tension.kicad_sch)
- added sheet Cond_Capt_Tension_Ph2 (Cond_Capt_Tension.kicad_sch)
- added sheet Cond_Capt_Tension_Ph3 (Cond_Capt_Tension.kicad_sch)
- added sheet Cond_Capt_Tension_Ph4 (Cond_Capt_Tension.kicad_sch)
- moved on the sheet: C1, C10, C11, C12, C13, C14, C2, C3, C4, C5, C6, C7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

Commit message: modif
Parts:
- added D2: LED_Orange, LED_SMD:LED_0603_1608Metric_Pad1.05x0.95mm_HandSolder, symbol Device:LED_Small
- added F1: Fuse, symbol Device:Fuse
- added H1, H2, H3, H4, H5, H6, H7, H8: MountingHole, symbol Mechanical:MountingHole
- added J4_Neutre1: Conn_01x01, Connector:Banana_Cliff_FCR7350B_S16N-PC_Horizontal, symbol Connector_Generic:Conn_01x01
- added R2: 1k, Resistor_SMD:R_0805_2012Metric_Pad1.20x1.40mm_HandSolder, symbol Device:R
- added TP1: TestPoint, symbol Connector:TestPoint
- C1, C2: value 10uF -> 10u; footprint (none) -> Capacitor_SMD:C_0805_2012Metric_Pad1.18x1.45mm_HandSolder
- C10, C11, C13, C14, C3, C4, C6, C7, C8, C9: value 0.1uF -> 0.1u; footprint (none) -> Capacitor_SMD:C_0805_2012Metric_Pad1.18x1.45mm_HandSolder
- C12, C5: value C -> 0.1u; footprint (none) -> Capacitor_SMD:C_0805_2012Metric_Pad1.18x1.45mm_HandSolder
- D1: value LED_Small -> LED_Green; footprint (none) -> LED_SMD:LED_0603_1608Metric_Pad1.05x0.95mm_HandSolder
- D3: renamed from D2; value LED_Small -> LED_Green; footprint (none) -> LED_SMD:LED_0603_1608Metric_Pad1.05x0.95mm_HandSolder
- R1: footprint (none) -> Resistor_SMD:R_0805_2012Metric_Pad1.20x1.40mm_HandSolder
- R3: renamed from R2; footprint (none) -> Resistor_SMD:R_0805_2012Metric_Pad1.20x1.40mm_HandSolder
- U3, U4, U5, U6, U7, U8: footprint (none) -> Package_SO:SOIC-8_3.9x4.9mm_P1.27mm
- renumbered J1_Vphase4 to J1_Vphase1, J1_Vphase1 to J1_Vphase2, J1_Vphase2 to J1_Vphase4
Connections:
- net +3V3: now also R2.1
- net GND: now also D2.1 (K), TP1.1
- net at U1.2 (AC(L)): now also F1.1; no longer J5_Ph_230V1.1 (Pin_1)
- new net: F1.2, J5_Ph_230V1.1 (Pin_1)
- new net: D2.2 (A), R2.2
- new net Neutre: J4_Neutre1.1 (Pin_1)
Other:
- sheet Cond_Capt_Tension_Ph1 ports: added J_conn_N; removed none
- sheet Cond_Capt_Tension_Ph2 ports: added J_conn_N; removed none
- sheet Cond_Capt_Tension_Ph3 ports: added J_conn_N; removed none
- sheet Cond_Capt_Tension_Ph4 ports: added J_conn_N; removed none
- moved on the sheet: C1, C10, C11, C12, C13, C14, C2, C3, C4, C5, C6, C7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

Commit message: modif
Parts:
- removed H1, H2, H3, H4, H5, H6, H7, H8: MountingHole, symbol Mechanical:MountingHole
- removed J1_Vphase1: Conn_01x01, Connector:Banana_Cliff_FCR7350B_S16N-PC_Horizontal, symbol Connector_Generic:Conn_01x01
- removed TP1: TestPoint, symbol Connector:TestPoint
- added H1, H2, H3, H4, H5, H6, H7, H8: MountingHole_Pad, MountingHole:MountingHole_3.2mm_M3_Pad, symbol Mechanical:MountingHole_Pad
- added JP1, JP2, JP3, JP4: SolderJumper_2_Open, Jumper:SolderJumper-2_P1.3mm_Open_TrianglePad1.0x1.5mm, symbol Jumper:SolderJumper_2_Open
- C1, C10, C11, C12, C13, C14, C2, C3, C4, C5, C6, C7, C8, C9: footprint Capacitor_SMD:C_0805_2012Metric_Pad1.18x1.45mm_HandSolder -> Capacitor_SMD:C_0603_1608Metric_Pad1.08x0.95mm_HandSolder
- F1: footprint (none) -> Library.pretty_Porte_Fusible:Porte_Fusible_PC1E
- R1: footprint Resistor_SMD:R_0805_2012Metric_Pad1.20x1.40mm_HandSolder -> Resistor_SMD:R_0603_1608Metric_Pad0.98x0.95mm_HandSolder
- R2: renamed from R3; footprint Resistor_SMD:R_0805_2012Metric_Pad1.20x1.40mm_HandSolder -> Resistor_SMD:R_0603_1608Metric_Pad0.98x0.95mm_HandSolder
- R3: renamed from R2; footprint Resistor_SMD:R_0805_2012Metric_Pad1.20x1.40mm_HandSolder -> Resistor_SMD:R_0603_1608Metric_Pad0.98x0.95mm_HandSolder
- renumbered D3 to D2, D2 to D3, J1_Vphase2 to J1_Vphase1, J1_Vphase3 to J1_Vphase2, J1_Vphase4 to J1_Vphase3
Connections:
- net +15V: now also JP1.2 (B); no longer R1.2, U1.6 (Vout1)
- net +3V3: now also JP4.1 (A); no longer R3.1
- net -15V: now also JP3.2 (B); no longer R2.1, U1.4 (Vout2)
- net GND: now also H1.1, H2.1, H3.1, H4.1, H5.1, H6.1, H7.1, H8.1, JP2.2 (B); no longer U1.5 (Comm)
- new net: JP3.1 (A), R2.1, U1.4 (Vout2)
- new net: JP2.1 (A), U1.5 (Comm)
- new net: JP1.1 (A), R1.2, U1.6 (Vout1)
- new net: JP4.2 (B), R3.1
- no-connect marks 0 -> 6
Other:
- removed sheet Cond_Capt_Tension_Ph4
- moved on the sheet: C1, C2, D1, D2, D3, F1, J5_Ph_230V1, J6_Neutre_230V1, R1, R2, R3, U1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

Commit message: modif
Parts:
- removed U3, U4, U5, U6, U7, U8: OP275, Package_SO:SOIC-8_3.9x4.9mm_P1.27mm, symbol Amplifier_Operational:OP275
- C1: value 10u -> 0.1u
- P1: footprint (none) -> Library.pretty_Dsub_15_Female:Dsub_15_Female_E

Commit message: modif
Parts:
- renumbered J1_Vphase1 to JB1, J1_Vphase2 to JB2, J1_Vphase3 to JB3, J4_Neutre1 to JB4, J5_Ph_230V1 to JB5, J6_Neutre_230V1 to JB6
Changed lines of the file:
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@@
 		(dnp no)
 		(fields_autoplaced yes)
-		(property "Reference" "J5_Ph_230V1"
+		(property "Reference" "JB5"
 			(at 87.63 88.9 0)
 			(effects
@@
 			(project "Kicad"
 				(path "/16213bc9-ed22-4e8b-8e21-f5cd88729472"
-					(reference "J5_Ph_230V1")
+					(reference "JB5")
 					(unit 1)
 				)
@@
 		(on_board yes)
 		(dnp no)
-		(property "Reference" "J6_Neutre_230V1"
+		(property "Reference" "JB6"
 			(at 88.138 103.632 0)
 			(effects
@@
 			(project "Kicad"
 				(path "/16213bc9-ed22-4e8b-8e21-f5cd88729472"
-					(reference "J6_Neutre_230V1")
+					(reference "JB6")
 					(unit 1)
 				)
@@
 		(dnp no)
 		(fields_autoplaced yes)
-		(property "Reference" "J1_Vphase1"
+		(property "Reference" "JB1"
 			(at 25.4 19.05 0)
 			(effects
@@
 			(project "Kicad"
 				(path "/16213bc9-ed22-4e8b-8e21-f5cd88729472"
-					(reference "J1_Vphase1")
+					(reference "JB1")
 					(unit 1)
 				)
@@
 		(on_board yes)
 		(dnp no)
-		(property "Reference" "J4_Neutre1"
+		(property "Reference" "JB4"
 			(at 26.416 71.12 0)
 			(effects
@@
 			(project "Kicad"
 				(path "/16213bc9-ed22-4e8b-8e21-f5cd88729472"
-					(reference "J4_Neutre1")
+					(reference "JB4")
 					(unit 1)
 				)
@@
 		(dnp no)
 		(fields_autoplaced yes)
-		(property "Reference" "J1_Vphase3"
+		(property "Reference" "JB3"
 			(at 151.13 19.05 0)
 			(effects
@@
 			(project "Kicad"
 				(path "/16213bc9-ed22-4e8b-8e21-f5cd88729472"
-					(reference "J1_Vphase3")
+					(reference "JB3")
 					(unit 1)
 				)
@@
 		(dnp no)
 		(fields_autoplaced yes)
-		(property "Reference" "J1_Vphase2"
+		(property "Reference" "JB2"
 			(at 88.9 19.05 0)
 			(effects
@@
 			(project "Kicad"
 				(path "/16213bc9-ed22-4e8b-8e21-f5cd88729472"
-					(reference "J1_Vphase2")
+					(reference "JB2")
 					(unit 1)
 				)
