File: Hardware/Kicad_Carte_Acquisition/Cond_Capt_Tension.kicad_sch (KiCad schematic)
At the start: 10 parts, among them J4_Neutre1 Conn_01x01, U11 LV25-P, U5 OP275

Commit message: modif
Parts:
- removed J4_Neutre1: Conn_01x01, Connector:Banana_Cliff_FCR7350B_S16N-PC_Horizontal, symbol Connector_Generic:Conn_01x01
- R20: renamed from R19; footprint (none) -> Resistor_SMD:R_0805_2012Metric_Pad1.20x1.40mm_HandSolder
- R22: renamed from R21; footprint (none) -> Resistor_SMD:R_0805_2012Metric_Pad1.20x1.40mm_HandSolder
- R23: renamed from R22; footprint (none) -> Resistor_SMD:R_0805_2012Metric_Pad1.20x1.40mm_HandSolder
- R24: renamed from R23; footprint (none) -> Resistor_SMD:R_0805_2012Metric_Pad1.20x1.40mm_HandSolder
- U5: footprint (none) -> Package_SO:SOIC-8_3.9x4.9mm_P1.27mm
- renumbered R20 to R21, TP5 to TP6, TP6 to TP7
Connections:
- net J_conn_N: now reaches U11.3 (HV-)
Other:
- moved on the sheet: TP7
Changed lines of the file:
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@@
+	)
+	(junction
+		(at 234.95 72.39)
+		(diameter 0)
+		(color 0 0 0 0)
 	)
 	(junction
@@
 	(wire
 		(pts
+			(xy 234.95 72.39) (xy 242.57 72.39)
+		)
+		(stroke
+			(width 0)
+			(type default)
+		)
+	)
+	(wire
+		(pts
 			(xy 194.31 81.28) (xy 194.31 69.85)
 		)
@@
 	(wire
 		(pts
-			(xy 228.6 72.39) (xy 242.57 72.39)
+			(xy 228.6 72.39) (xy 234.95 72.39)
 		)
 		(stroke
@@
 				(hide yes)
 			)
+		)
+	)
+	(hierarchical_label "J_conn_N"
+		(shape input)
+		(at 115.57 90.17 180)
+		(fields_autoplaced yes)
+		(effects
+			(font
+				(size 1.27 1.27)
+			)
+			(justify right)
 		)
 	)
@@
 			)
 		)
-		(property "Footprint" ""
+		(property "Footprint" "Package_SO:SOIC-8_3.9x4.9mm_P1.27mm"
 			(at 184.15 69.85 0)
 			(effects
@@
 		(dnp no)
 		(fields_autoplaced yes)
-		(property "Reference" "R19"
+		(property "Reference" "R20"
 			(at 210.82 62.2299 0)
 			(effects
@@
 			)
 		)
-		(property "Footprint" ""
+		(property "Footprint" "Resistor_SMD:R_0805_2012Metric_Pad1.20x1.40mm_HandSolder"
 			(at 206.502 63.5 90)
 			(effects
@@
 			(project "Kicad"
 				(path "/16213bc9-ed22-4e8b-8e21-f5cd88729472/6ad54b17-3074-46c7-a14e-186ca26a6b2a"
-					(reference "R19")
+					(reference "R20")
 					(unit 1)
 				)
 				(path "/16213bc9-ed22-4e8b-8e21-f5cd88729472/ce9e0ffa-1841-4859-8d91-ed38360d7046"
-					(reference "R24")
+					(reference "R25")
 					(unit 1)
 				)
 				(path "/16213bc9-ed22-4e8b-8e21-f5cd88729472/7501b4d2-8ff2-45d5-930d-9dfb06f579e6"
-					(reference "R29")
+					(reference "R30")
 					(unit 1)
 				)
 				(path "/16213bc9-ed22-4e8b-8e21-f5cd88729472/b9fff193-61ef-4ba4-92e4-50182fcd544c"
-					(reference "R34")
+					(reference "R35")
 					(unit 1)
 				)
@@
 			)
 		)
-		(property "Footprint" ""
+		(property "Footprint" "Package_SO:SOIC-8_3.9x4.9mm_P1.27mm"
 			(at 218.44 72.39 0)
 			(effects
@@
 	(symbol
 		(lib_id "Connector:TestPoint")
-		(at 228.6 72.39 0)
+		(at 234.95 72.39 0)
 		(unit 1)
 		(exclude_from_sim no)
@@
 		(on_board yes)
 		(dnp no)
-		(property "Reference" "TP6"
-			(at 229.616 69.088 0)
+		(property "Reference" "TP7"
+			(at 235.966 69.088 0)
 			(effects
 				(font
@@
 		)
 		(property "Value" "TestPoint"
-			(at 226.822 66.04 0)
+			(at 233.172 66.04 0)
 			(effects
 				(font
@@
 		)
 		(property "Footprint" ""
-			(at 233.68 72.39 0)
+			(at 240.03 72.39 0)
 			(effects
 				(font
@@
 		)
 		(property "Datasheet" "~"
-			(at 233.68 72.39 0)
+			(at 240.03 72.39 0)
 			(effects
 				(font
@@
 		)
 		(property "Description" "test point"
-			(at 228.6 72.39 0)
+			(at 234.95 72.39 0)
 			(effects
 				(font
@@
 			(project "Kicad"
 				(path "/16213bc9-ed22-4e8b-8e21-f5cd88729472/6ad54b17-3074-46c7-a14e-186ca26a6b2a"
-					(reference "TP6")
+					(reference "TP7")
 					(unit 1)
 				)
 				(path "/16213bc9-ed22-4e8b-8e21-f5cd88729472/ce9e0ffa-1841-4859-8d91-ed38360d7046"
-					(reference "TP8")
+					(reference "TP9")
 					(unit 1)
 				)
 				(path "/16213bc9-ed22-4e8b-8e21-f5cd88729472/7501b4d2-8ff2-45d5-930d-9dfb06f579e6"
-					(reference "TP10")
+					(reference "TP11")
 					(unit 1)
 				)
 				(path "/16213bc9-ed22-4e8b-8e21-f5cd88729472/b9fff193-61ef-4ba4-92e4-50182fcd544c"
-					(reference "TP12")
+					(reference "TP13")
 					(unit 1)
 				)
@@
 		(dnp no)
 		(fields_autoplaced yes)
-		(property "Reference" "R23"
+		(property "Reference" "R24"
 			(at 184.15 74.93 90)
 			(effects
@@
 			)
 		)
-		(property "Footprint" ""
+		(property "Footprint" "Resistor_SMD:R_0805_2012Metric_Pad1.20x1.40mm_HandSolder"
 			(at 184.15 83.058 90)
 			(effects
@@
 			(project "Kicad"
 				(path "/16213bc9-ed22-4e8b-8e21-f5cd88729472/6ad54b17-3074-46c7-a14e-186ca26a6b2a"
-					(reference "R23")
+					(reference "R24")
 					(unit 1)
 				)
 				(path "/16213bc9-ed22-4e8b-8e21-f5cd88729472/ce9e0ffa-1841-4859-8d91-ed38360d7046"
-					(reference "R28")
+					(reference "R29")
 					(unit 1)
 				)
 				(path "/16213bc9-ed22-4e8b-8e21-f5cd88729472/7501b4d2-8ff2-45d5-930d-9dfb06f579e6"
-					(reference "R33")
+					(reference "R34")
 					(unit 1)
 				)
 				(path "/16213bc9-ed22-4e8b-8e21-f5cd88729472/b9fff193-61ef-4ba4-92e4-50182fcd544c"
-					(reference "R38")
-					(unit 1)
-				)
-			)
-		)
-	)
-	(symbol
-		(lib_id "Connector_Generic:Conn_01x01")
-		(at 110.49 90.17 180)
-		(unit 1)
-		(exclude_from_sim no)
-		(in_bom yes)
-		(on_board yes)
-		(dnp no)
-		(fields_autoplaced yes)
-		(property "Reference" "J4_Neutre1"
-			(at 110.49 83.82 0)
-			(effects
-				(font
-					(size 1.27 1.27)
-				)
-			)
-		)
-		(property "Value" "Conn_01x01"
-			(at 110.49 86.36 0)
-			(effects
-				(font
-					(size 1.27 1.27)
-				)
-			)
-		)
-		(property "Footprint" "Connector:Banana_Cliff_FCR7350B_S16N-PC_Horizontal"
-			(at 110.49 90.17 0)
-			(effects
-				(font
-					(size 1.27 1.27)
-				)
-				(hide yes)
-			)
-		)
-		(property "Datasheet" "~"
-			(at 110.49 90.17 0)
-			(effects
-				(font
-					(size 1.27 1.27)
-				)
-				(hide yes)
-			)
-		)
-		(property "Description" "Generic connector, single row, 01x01, script generated (kicad-library-utils/schlib/autogen/connector/)"
-			(at 110.49 90.17 0)
-			(effects
-				(font
-					(size 1.27 1.27)
-				)
-				(hide yes)
-			)
-		)
-		(pin "1"
-		)
-		(instances
-			(project "Kicad"
-				(path "/16213bc9-ed22-4e8b-8e21-f5cd88729472/6ad54b17-3074-46c7-a14e-186ca26a6b2a"
-					(reference "J4_Neutre1")
-					(unit 1)
-				)
-				(path "/16213bc9-ed22-4e8b-8e21-f5cd88729472/ce9e0ffa-1841-4859-8d91-ed38360d7046"
-					(reference "J4_Neutre2")
-					(unit 1)
-				)
-				(path "/16213bc9-ed22-4e8b-8e21-f5cd88729472/7501b4d2-8ff2-45d5-930d-9dfb06f579e6"
-					(reference "J4_Neutre3")
-					(unit 1)
-				)
-				(path "/16213bc9-ed22-4e8b-8e21-f5cd88729472/b9fff193-61ef-4ba4-92e4-50182fcd544c"
-					(reference "J4_Neutre4")
+					(reference "R39")
 					(unit 1)
 				)
@@
 		(on_board yes)
 		(dnp no)
-		(property "Reference" "TP5"
+		(property "Reference" "TP6"
 			(at 169.418 64.262 0)
 			(effects
@@
 			(project "Kicad"
 				(path "/16213bc9-ed22-4e8b-8e21-f5cd88729472/6ad54b17-3074-46c7-a14e-186ca26a6b2a"
-					(reference "TP5")
+					(reference "TP6")
 					(unit 1)
 				)
 				(path "/16213bc9-ed22-4e8b-8e21-f5cd88729472/ce9e0ffa-1841-4859-8d91-ed38360d7046"
-					(reference "TP7")
+					(reference "TP8")
 					(unit 1)
 				)
 				(path "/16213bc9-ed22-4e8b-8e21-f5cd88729472/7501b4d2-8ff2-45d5-930d-9dfb06f579e6"
-					(reference "TP9")
+					(reference "TP10")
 					(unit 1)
 				)
 				(path "/16213bc9-ed22-4e8b-8e21-f5cd88729472/b9fff193-61ef-4ba4-92e4-50182fcd544c"
-					(reference "TP11")
+					(reference "TP12")
 					(unit 1)
 				)
@@
 		(dnp no)
 		(fields_autoplaced yes)
-		(property "Reference" "R20"
+		(property "Reference" "R21"
 			(at 127 58.42 90)
 			(effects
@@
 			(project "Kicad"
 				(path "/16213bc9-ed22-4e8b-8e21-f5cd88729472/6ad54b17-3074-46c7-a14e-186ca26a6b2a"
-					(reference "R20")
+					(reference "R21")
 					(unit 1)
 				)
 				(path "/16213bc9-ed22-4e8b-8e21-f5cd88729472/ce9e0ffa-1841-4859-8d91-ed38360d7046"
-					(reference "R25")
+					(reference "R26")
 					(unit 1)
 				)
 				(path "/16213bc9-ed22-4e8b-8e21-f5cd88729472/7501b4d2-8ff2-45d5-930d-9dfb06f579e6"
-					(reference "R30")
+					(reference "R31")
 					(unit 1)
 				)
 				(path "/16213bc9-ed22-4e8b-8e21-f5cd88729472/b9fff193-61ef-4ba4-92e4-50182fcd544c"
-					(reference "R35")
+					(reference "R36")
 					(unit 1)
 				)
@@
 		(dnp no)
 		(fields_autoplaced yes)
-		(property "Reference" "R22"
+		(property "Reference" "R23"
 			(at 157.48 73.6599 0)
 			(effects
@@
 			)
 		)
-		(property "Footprint" ""
+		(property "Footprint" "Resistor_SMD:R_0805_2012Metric_Pad1.20x1.40mm_HandSolder"
 			(at 156.718 74.93 90)
 			(effects
@@
 			(project "Kicad"
 				(path "/16213bc9-ed22-4e8b-8e21-f5cd88729472/6ad54b17-3074-46c7-a14e-186ca26a6b2a"
-					(reference "R22")
+					(reference "R23")
 					(unit 1)
 				)
 				(path "/16213bc9-ed22-4e8b-8e21-f5cd88729472/ce9e0ffa-1841-4859-8d91-ed38360d7046"
-					(reference "R27")
+					(reference "R28")
 					(unit 1)
 				)
 				(path "/16213bc9-ed22-4e8b-8e21-f5cd88729472/7501b4d2-8ff2-45d5-930d-9dfb06f579e6"
-					(reference "R32")
+					(reference "R33")
 					(unit 1)
 				)
 				(path "/16213bc9-ed22-4e8b-8e21-f5cd88729472/b9fff193-61ef-4ba4-92e4-50182fcd544c"
-					(reference "R37")
+					(reference "R38")
 					(unit 1)
 				)
@@
 		(dnp no)
 		(fields_autoplaced yes)
-		(property "Reference" "R21"
+		(property "Reference" "R22"
 			(at 200.66 63.5 90)
 			(effects
@@
 			)
 		)
-		(property "Footprint" ""
+		(property "Footprint" "Resistor_SMD:R_0805_2012Metric_Pad1.20x1.40mm_HandSolder"
 			(at 200.66 71.628 90)
 			(effects
@@
 			(project "Kicad"
 				(path "/16213bc9-ed22-4e8b-8e21-f5cd88729472/6ad54b17-3074-46c7-a14e-186ca26a6b2a"
-					(reference "R21")
+					(reference "R22")
 					(unit 1)
 				)
 				(path "/16213bc9-ed22-4e8b-8e21-f5cd88729472/ce9e0ffa-1841-4859-8d91-ed38360d7046"
-					(reference "R26")
+					(reference "R27")
 					(unit 1)
 				)
 				(path "/16213bc9-ed22-4e8b-8e21-f5cd88729472/7501b4d2-8ff2-45d5-930d-9dfb06f579e6"
-					(reference "R31")
+					(reference "R32")
 					(unit 1)
 				)
 				(path "/16213bc9-ed22-4e8b-8e21-f5cd88729472/b9fff193-61ef-4ba4-92e4-50182fcd544c"
-					(reference "R36")
-					(unit 1)
-				)
+					(reference "R37")
+					(unit 1)
+				)

Commit message: modif
Parts:
- removed TP6, TP7: TestPoint, symbol Connector:TestPoint
- added JP10, JP9: SolderJumper_2_Open, Jumper:SolderJumper-2_P1.3mm_Open_TrianglePad1.0x1.5mm, symbol Jumper:SolderJumper_2_Open
- R20, R22, R23, R24: footprint Resistor_SMD:R_0805_2012Metric_Pad1.20x1.40mm_HandSolder -> Resistor_SMD:R_0603_1608Metric_Pad0.98x0.95mm_HandSolder
- R21: footprint (none) -> Library.pretty_R_4527_M11470:R_4527_M11470E
- renumbered U11 to U10
Connections:
- net Vphase_out: now also JP10.2 (B); no longer U5.6 (-), U5.7
- net at R23.2, U10.4 (M): now also JP9.1 (A); no longer U5.3 (+)
- new net: JP9.2 (B), U5.3 (+)
- new net: JP10.1 (A), U5.6 (-), U5.7

Commit message: modif
Parts:
- added unit 3 of U7
- renumbered U5 to U7, U10 to U8
Connections:
- net +15V: now also U7.8 (V+)
- new net -15V: U7.4 (V-)
Changed lines of the file:
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@@
+	(wire
+		(pts
+			(xy 237.49 33.02) (xy 237.49 34.29)
+		)
+		(stroke
+			(width 0)
+			(type default)
+		)
+	)
 	(wire
 		(pts
@@
 	(wire
 		(pts
+			(xy 237.49 50.8) (xy 237.49 49.53)
+		)
+		(stroke
+			(width 0)
+			(type default)
+		)
+	)
+	(wire
+		(pts
 			(xy 187.96 81.28) (xy 194.31 81.28)
 		)
@@
 	(wire
 		(pts
+			(xy 237.49 50.8) (xy 246.38 50.8)
+		)
+		(stroke
+			(width 0)
+			(type default)
+		)
+	)
+	(wire
+		(pts
 			(xy 208.28 69.85) (xy 210.82 69.85)
 		)
@@
 	(wire
 		(pts
+			(xy 245.11 33.02) (xy 237.49 33.02)
+		)
+		(stroke
+			(width 0)
+			(type default)
+		)
+	)
+	(wire
+		(pts
 			(xy 194.31 81.28) (xy 194.31 69.85)
 		)
@@
 			(width 0)
 			(type default)
+		)
+	)
+	(global_label "+15V"
+		(shape input)
+		(at 245.11 33.02 0)
+		(fields_autoplaced yes)
+		(effects
+			(font
+				(size 1.27 1.27)
+			)
+			(justify left)
+		)
+		(property "Intersheetrefs" "${INTERSHEET_REFS}"
+			(at 253.1752 33.02 0)
+			(effects
+				(font
+					(size 1.27 1.27)
+				)
+				(justify left)
+				(hide yes)
+			)
 		)
 	)
@@
 				)
 				(justify right)
+				(hide yes)
+			)
+		)
+	)
+	(global_label "-15V"
+		(shape input)
+		(at 246.38 50.8 0)
+		(fields_autoplaced yes)
+		(effects
+			(font
+				(size 1.27 1.27)
+			)
+			(justify left)
+		)
+		(property "Intersheetrefs" "${INTERSHEET_REFS}"
+			(at 254.4452 50.8 0)
+			(effects
+				(font
+					(size 1.27 1.27)
+				)
+				(justify left)
 				(hide yes)
 			)
@@
 		(dnp no)
 		(fields_autoplaced yes)
-		(property "Reference" "U5"
+		(property "Reference" "U7"
 			(at 184.15 59.69 0)
 			(effects
@@
 			(project "Kicad"
 				(path "/16213bc9-ed22-4e8b-8e21-f5cd88729472/6ad54b17-3074-46c7-a14e-186ca26a6b2a"
-					(reference "U5")
+					(reference "U7")
 					(unit 1)
 				)
 				(path "/16213bc9-ed22-4e8b-8e21-f5cd88729472/ce9e0ffa-1841-4859-8d91-ed38360d7046"
-					(reference "U6")
+					(reference "U9")
 					(unit 1)
 				)
 				(path "/16213bc9-ed22-4e8b-8e21-f5cd88729472/7501b4d2-8ff2-45d5-930d-9dfb06f579e6"
-					(reference "U7")
+					(reference "U11")
 					(unit 1)
 				)
@@
 		(dnp no)
 		(fields_autoplaced yes)
-		(property "Reference" "U5"
+		(property "Reference" "U7"
 			(at 218.44 62.23 0)
 			(effects
@@
 			(project "Kicad"
 				(path "/16213bc9-ed22-4e8b-8e21-f5cd88729472/6ad54b17-3074-46c7-a14e-186ca26a6b2a"
-					(reference "U5")
+					(reference "U7")
 					(unit 2)
 				)
 				(path "/16213bc9-ed22-4e8b-8e21-f5cd88729472/ce9e0ffa-1841-4859-8d91-ed38360d7046"
-					(reference "U6")
+					(reference "U9")
 					(unit 2)
 				)
 				(path "/16213bc9-ed22-4e8b-8e21-f5cd88729472/7501b4d2-8ff2-45d5-930d-9dfb06f579e6"
-					(reference "U7")
+					(reference "U11")
 					(unit 2)
 				)
@@
 		(on_board yes)
 		(dnp no)
-		(property "Reference" "U10"
+		(property "Reference" "U8"
 			(at 151.638 58.42 0)
 			(effects
@@
 			(project "Kicad"
 				(path "/16213bc9-ed22-4e8b-8e21-f5cd88729472/6ad54b17-3074-46c7-a14e-186ca26a6b2a"
+					(reference "U8")
+					(unit 1)
+				)
+				(path "/16213bc9-ed22-4e8b-8e21-f5cd88729472/ce9e0ffa-1841-4859-8d91-ed38360d7046"
 					(reference "U10")
-					(unit 1)
-				)
-				(path "/16213bc9-ed22-4e8b-8e21-f5cd88729472/ce9e0ffa-1841-4859-8d91-ed38360d7046"
-					(reference "U11")
 					(unit 1)
 				)
@@
 				)
 			)
+		)
+	)
+	(symbol
+		(lib_id "Amplifier_Operational:OP275")
+		(at 240.03 41.91 0)
+		(unit 3)
+		(exclude_from_sim no)
+		(in_bom yes)
+		(on_board yes)
+		(dnp no)
+		(property "Reference" "U7"
+			(at 239.268 40.386 0)
+			(effects
+				(font
+					(size 1.27 1.27)
+				)
+				(justify left)
+			)
+		)
+		(property "Value" "OP275"
+			(at 239.268 42.926 0)
+			(effects
+				(font
+					(size 1.27 1.27)
+				)
+				(justify left)
+			)
+		)
+		(property "Footprint" "Package_SO:SOIC-8_3.9x4.9mm_P1.27mm"
+			(at 240.03 41.91 0)
+			(effects
+				(font
+					(size 1.27 1.27)
+				)
+				(hide yes)
+			)
+		)
+		(property "Datasheet" "https://www.analog.com/media/en/technical-documentation/data-sheets/OP275.pdf"
+			(at 240.03 41.91 0)
+			(effects
+				(font
+					(size 1.27 1.27)
+				)
+				(hide yes)
+			)
+		)
+		(property "Description" "Dual Bipolar/JFET, Audio Operational Amplifier, DIP-8/SOIC-8"
+			(at 240.03 41.91 0)
+			(effects
+				(font
+					(size 1.27 1.27)
+				)
+				(hide yes)
+			)
+		)
+		(pin "3"
+		)
+		(pin "7"
+		)
+		(pin "2"
+		)
+		(pin "6"
+		)
+		(pin "4"
+		)
+		(pin "8"
+		)
+		(pin "5"
+		)
+		(pin "1"
+		)
+		(instances
+			(project "Kicad"
+				(path "/16213bc9-ed22-4e8b-8e21-f5cd88729472/6ad54b17-3074-46c7-a14e-186ca26a6b2a"
+					(reference "U7")
+					(unit 3)
+				)
+				(path "/16213bc9-ed22-4e8b-8e21-f5cd88729472/ce9e0ffa-1841-4859-8d91-ed38360d7046"
+					(reference "U9")
+					(unit 3)
+				)
+				(path "/16213bc9-ed22-4e8b-8e21-f5cd88729472/7501b4d2-8ff2-45d5-930d-9dfb06f579e6"
+					(reference "U11")
+					(unit 3)
+				)
+			)

Commit message: modif
Connections:
- net +15V: no longer U8.6 (V-)
- net -15V: now also U8.6 (V-)
Changed lines of the file:
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@@
 		)
 	)
-	(global_label "+15V"
+	(global_label "-15V"
 		(shape input)
 		(at 140.97 88.9 180)
