File: Hardware/Kicad_Carte_Acquisition/Conditionnement_capteur.kicad_sch (KiCad schematic)
At the start: 7 parts, among them J1 Conn_Coaxial, U13 OP275

Commit message: modif
Parts:
- R3: renamed from R35; value R -> 1k
- R4: renamed from R34; value 11k -> 1k
- R5: renamed from R32; value R -> 8.25k
- R6: renamed from R33; value R -> 1k
- renumbered TP11 to TP1, U13 to U3
Other:
- moved on the sheet: TP1

Commit message: modif
Parts:
- R4: renamed from R3; footprint (none) -> Resistor_SMD:R_0805_2012Metric_Pad1.20x1.40mm_HandSolder
- R5: renamed from R4; footprint (none) -> Resistor_SMD:R_0805_2012Metric_Pad1.20x1.40mm_HandSolder
- R6: renamed from R5; footprint (none) -> Resistor_SMD:R_0805_2012Metric_Pad1.20x1.40mm_HandSolder
- R7: renamed from R6; footprint (none) -> Resistor_SMD:R_0805_2012Metric_Pad1.20x1.40mm_HandSolder
- U3: footprint (none) -> Package_SO:SOIC-8_3.9x4.9mm_P1.27mm
- renumbered TP1 to TP2
Changed lines of the file:
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@@
 			)
 		)
-		(property "Footprint" ""
+		(property "Footprint" "Package_SO:SOIC-8_3.9x4.9mm_P1.27mm"
 			(at 151.13 95.25 0)
 			(effects
@@
 		(dnp no)
 		(fields_autoplaced yes)
-		(property "Reference" "R6"
+		(property "Reference" "R7"
 			(at 163.83 109.2199 0)
 			(effects
@@
 			)
 		)
-		(property "Footprint" ""
+		(property "Footprint" "Resistor_SMD:R_0805_2012Metric_Pad1.20x1.40mm_HandSolder"
 			(at 159.512 110.49 90)
 			(effects
@@
 			(project "Kicad"
 				(path "/16213bc9-ed22-4e8b-8e21-f5cd88729472/72d653c3-8f6f-4150-b7cd-d5c98c703715"
-					(reference "R6")
-					(unit 1)
-				)
-				(path "/16213bc9-ed22-4e8b-8e21-f5cd88729472/a83cc724-240f-4e24-86d0-fe129e515c9d"
-					(reference "R10")
-					(unit 1)
-				)
-				(path "/16213bc9-ed22-4e8b-8e21-f5cd88729472/f65a2aaa-bdb9-4087-a40a-8b8d146426dc"
-					(reference "R14")
-					(unit 1)
-				)
-				(path "/16213bc9-ed22-4e8b-8e21-f5cd88729472/9b53e793-8acb-49d6-9671-6c75b365109f"
-					(reference "R18")
+					(reference "R7")
+					(unit 1)
+				)
+				(path "/16213bc9-ed22-4e8b-8e21-f5cd88729472/a83cc724-240f-4e24-86d0-fe129e515c9d"
+					(reference "R11")
+					(unit 1)
+				)
+				(path "/16213bc9-ed22-4e8b-8e21-f5cd88729472/f65a2aaa-bdb9-4087-a40a-8b8d146426dc"
+					(reference "R15")
+					(unit 1)
+				)
+				(path "/16213bc9-ed22-4e8b-8e21-f5cd88729472/9b53e793-8acb-49d6-9671-6c75b365109f"
+					(reference "R19")
 					(unit 1)
 				)
@@
 		(dnp no)
 		(fields_autoplaced yes)
-		(property "Reference" "R4"
+		(property "Reference" "R5"
 			(at 168.91 88.9 90)
 			(effects
@@
 			)
 		)
-		(property "Footprint" ""
+		(property "Footprint" "Resistor_SMD:R_0805_2012Metric_Pad1.20x1.40mm_HandSolder"
 			(at 168.91 93.472 90)
 			(effects
@@
 			(project "Kicad"
 				(path "/16213bc9-ed22-4e8b-8e21-f5cd88729472/72d653c3-8f6f-4150-b7cd-d5c98c703715"
-					(reference "R4")
-					(unit 1)
-				)
-				(path "/16213bc9-ed22-4e8b-8e21-f5cd88729472/a83cc724-240f-4e24-86d0-fe129e515c9d"
-					(reference "R8")
-					(unit 1)
-				)
-				(path "/16213bc9-ed22-4e8b-8e21-f5cd88729472/f65a2aaa-bdb9-4087-a40a-8b8d146426dc"
-					(reference "R12")
-					(unit 1)
-				)
-				(path "/16213bc9-ed22-4e8b-8e21-f5cd88729472/9b53e793-8acb-49d6-9671-6c75b365109f"
-					(reference "R16")
+					(reference "R5")
+					(unit 1)
+				)
+				(path "/16213bc9-ed22-4e8b-8e21-f5cd88729472/a83cc724-240f-4e24-86d0-fe129e515c9d"
+					(reference "R9")
+					(unit 1)
+				)
+				(path "/16213bc9-ed22-4e8b-8e21-f5cd88729472/f65a2aaa-bdb9-4087-a40a-8b8d146426dc"
+					(reference "R13")
+					(unit 1)
+				)
+				(path "/16213bc9-ed22-4e8b-8e21-f5cd88729472/9b53e793-8acb-49d6-9671-6c75b365109f"
+					(reference "R17")
 					(unit 1)
 				)
@@
 		(on_board yes)
 		(dnp no)
-		(property "Reference" "TP1"
+		(property "Reference" "TP2"
 			(at 204.978 91.948 0)
 			(effects
@@
 			(project "Kicad"
 				(path "/16213bc9-ed22-4e8b-8e21-f5cd88729472/72d653c3-8f6f-4150-b7cd-d5c98c703715"
-					(reference "TP1")
-					(unit 1)
-				)
-				(path "/16213bc9-ed22-4e8b-8e21-f5cd88729472/a83cc724-240f-4e24-86d0-fe129e515c9d"
 					(reference "TP2")
 					(unit 1)
 				)
-				(path "/16213bc9-ed22-4e8b-8e21-f5cd88729472/f65a2aaa-bdb9-4087-a40a-8b8d146426dc"
+				(path "/16213bc9-ed22-4e8b-8e21-f5cd88729472/a83cc724-240f-4e24-86d0-fe129e515c9d"
 					(reference "TP3")
 					(unit 1)
 				)
-				(path "/16213bc9-ed22-4e8b-8e21-f5cd88729472/9b53e793-8acb-49d6-9671-6c75b365109f"
+				(path "/16213bc9-ed22-4e8b-8e21-f5cd88729472/f65a2aaa-bdb9-4087-a40a-8b8d146426dc"
 					(reference "TP4")
+					(unit 1)
+				)
+				(path "/16213bc9-ed22-4e8b-8e21-f5cd88729472/9b53e793-8acb-49d6-9671-6c75b365109f"
+					(reference "TP5")
 					(unit 1)
 				)
@@
 			)
 		)
-		(property "Footprint" ""
+		(property "Footprint" "Package_SO:SOIC-8_3.9x4.9mm_P1.27mm"
 			(at 182.88 97.79 0)
 			(effects
@@
 		(dnp no)
 		(fields_autoplaced yes)
-		(property "Reference" "R3"
+		(property "Reference" "R4"
 			(at 176.53 86.3599 0)
 			(effects
@@
 			)
 		)
-		(property "Footprint" ""
+		(property "Footprint" "Resistor_SMD:R_0805_2012Metric_Pad1.20x1.40mm_HandSolder"
 			(at 172.212 87.63 90)
 			(effects
@@
 			(project "Kicad"
 				(path "/16213bc9-ed22-4e8b-8e21-f5cd88729472/72d653c3-8f6f-4150-b7cd-d5c98c703715"
-					(reference "R3")
-					(unit 1)
-				)
-				(path "/16213bc9-ed22-4e8b-8e21-f5cd88729472/a83cc724-240f-4e24-86d0-fe129e515c9d"
-					(reference "R7")
-					(unit 1)
-				)
-				(path "/16213bc9-ed22-4e8b-8e21-f5cd88729472/f65a2aaa-bdb9-4087-a40a-8b8d146426dc"
-					(reference "R11")
-					(unit 1)
-				)
-				(path "/16213bc9-ed22-4e8b-8e21-f5cd88729472/9b53e793-8acb-49d6-9671-6c75b365109f"
-					(reference "R15")
+					(reference "R4")
+					(unit 1)
+				)
+				(path "/16213bc9-ed22-4e8b-8e21-f5cd88729472/a83cc724-240f-4e24-86d0-fe129e515c9d"
+					(reference "R8")
+					(unit 1)
+				)
+				(path "/16213bc9-ed22-4e8b-8e21-f5cd88729472/f65a2aaa-bdb9-4087-a40a-8b8d146426dc"
+					(reference "R12")
+					(unit 1)
+				)
+				(path "/16213bc9-ed22-4e8b-8e21-f5cd88729472/9b53e793-8acb-49d6-9671-6c75b365109f"
+					(reference "R16")
 					(unit 1)
 				)
@@
 		(dnp no)
 		(fields_autoplaced yes)
-		(property "Reference" "R5"
+		(property "Reference" "R6"
 			(at 163.83 99.0599 0)
 			(effects
@@
 			)
 		)
-		(property "Footprint" ""
+		(property "Footprint" "Resistor_SMD:R_0805_2012Metric_Pad1.20x1.40mm_HandSolder"
 			(at 159.512 100.33 90)
 			(effects
@@
 			(project "Kicad"
 				(path "/16213bc9-ed22-4e8b-8e21-f5cd88729472/72d653c3-8f6f-4150-b7cd-d5c98c703715"
-					(reference "R5")
-					(unit 1)
-				)
-				(path "/16213bc9-ed22-4e8b-8e21-f5cd88729472/a83cc724-240f-4e24-86d0-fe129e515c9d"
-					(reference "R9")
-					(unit 1)
-				)
-				(path "/16213bc9-ed22-4e8b-8e21-f5cd88729472/f65a2aaa-bdb9-4087-a40a-8b8d146426dc"
-					(reference "R13")
-					(unit 1)
-				)
-				(path "/16213bc9-ed22-4e8b-8e21-f5cd88729472/9b53e793-8acb-49d6-9671-6c75b365109f"
-					(reference "R17")
-					(unit 1)
-				)
+					(reference "R6")
+					(unit 1)
+				)
+				(path "/16213bc9-ed22-4e8b-8e21-f5cd88729472/a83cc724-240f-4e24-86d0-fe129e515c9d"
+					(reference "R10")
+					(unit 1)
+				)
+				(path "/16213bc9-ed22-4e8b-8e21-f5cd88729472/f65a2aaa-bdb9-4087-a40a-8b8d146426dc"
+					(reference "R14")
+					(unit 1)
+				)
+				(path "/16213bc9-ed22-4e8b-8e21-f5cd88729472/9b53e793-8acb-49d6-9671-6c75b365109f"
+					(reference "R18")
+					(unit 1)
+				)

Commit message: modif
Parts:
- removed TP2: TestPoint, symbol Connector:TestPoint
- added JP5: SolderJumper_2_Open, Jumper:SolderJumper-2_P1.3mm_Open_TrianglePad1.0x1.5mm, symbol Jumper:SolderJumper_2_Open
- R4, R5, R6, R7: footprint Resistor_SMD:R_0805_2012Metric_Pad1.20x1.40mm_HandSolder -> Resistor_SMD:R_0603_1608Metric_Pad0.98x0.95mm_HandSolder
Connections:
- net out: now also JP5.2 (B); no longer U3.6 (-), U3.7
- new net: JP5.1 (A), U3.6 (-), U3.7
Changed lines of the file:
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@@
 	(paper "A4")
-	(junction
-		(at 203.2 97.79)
-		(diameter 0)
-		(color 0 0 0 0)
-	)
 	(junction
 		(at 161.29 95.25)
@@
 	(wire
 		(pts
-			(xy 203.2 95.25) (xy 203.2 97.79)
-		)
-		(stroke
-			(width 0)
-			(type default)
-		)
-	)
-	(wire
-		(pts
-			(xy 214.63 97.79) (xy 203.2 97.79)
-		)
-		(stroke
-			(width 0)
-			(type default)
-		)
-	)
-	(wire
-		(pts
 			(xy 140.97 105.41) (xy 161.29 105.41)
 		)
@@
 	(wire
 		(pts
-			(xy 193.04 97.79) (xy 203.2 97.79)
-		)
-		(stroke
-			(width 0)
-			(type default)
-		)
-	)
-	(wire
-		(pts
 			(xy 175.26 104.14) (xy 193.04 104.14)
 		)
@@
 		(pts
 			(xy 193.04 104.14) (xy 193.04 97.79)
+		)
+		(stroke
+			(width 0)
+			(type default)
+		)
+	)
+	(wire
+		(pts
+			(xy 208.28 97.79) (xy 214.63 97.79)
+		)
+		(stroke
+			(width 0)
+			(type default)
+		)
+	)
+	(wire
+		(pts
+			(xy 193.04 97.79) (xy 200.66 97.79)
 		)
 		(stroke
@@
 		(dnp no)
 		(fields_autoplaced yes)
-		(property "Reference" "#PWR011"
+		(property "Reference" "#PWR013"
 			(at 161.29 123.19 0)
 			(effects
@@
 			(project "Kicad"
 				(path "/16213bc9-ed22-4e8b-8e21-f5cd88729472/72d653c3-8f6f-4150-b7cd-d5c98c703715"
-					(reference "#PWR011")
+					(reference "#PWR013")
 					(unit 1)
 				)
 				(path "/16213bc9-ed22-4e8b-8e21-f5cd88729472/a83cc724-240f-4e24-86d0-fe129e515c9d"
-					(reference "#PWR014")
+					(reference "#PWR016")
 					(unit 1)
 				)
 				(path "/16213bc9-ed22-4e8b-8e21-f5cd88729472/f65a2aaa-bdb9-4087-a40a-8b8d146426dc"
-					(reference "#PWR017")
+					(reference "#PWR019")
 					(unit 1)
 				)
 				(path "/16213bc9-ed22-4e8b-8e21-f5cd88729472/9b53e793-8acb-49d6-9671-6c75b365109f"
-					(reference "#PWR020")
+					(reference "#PWR022")
 					(unit 1)
 				)
@@
 				)
 				(path "/16213bc9-ed22-4e8b-8e21-f5cd88729472/f65a2aaa-bdb9-4087-a40a-8b8d146426dc"
+					(reference "U8")
+					(unit 1)
+				)
+				(path "/16213bc9-ed22-4e8b-8e21-f5cd88729472/9b53e793-8acb-49d6-9671-6c75b365109f"
 					(reference "U9")
-					(unit 1)
-				)
-				(path "/16213bc9-ed22-4e8b-8e21-f5cd88729472/9b53e793-8acb-49d6-9671-6c75b365109f"
-					(reference "U10")
 					(unit 1)
 				)
@@
 		(dnp no)
 		(fields_autoplaced yes)
-		(property "Reference" "#PWR010"
+		(property "Reference" "#PWR012"
 			(at 127 91.44 0)
 			(effects
@@
 			(project "Kicad"
 				(path "/16213bc9-ed22-4e8b-8e21-f5cd88729472/72d653c3-8f6f-4150-b7cd-d5c98c703715"
-					(reference "#PWR010")
+					(reference "#PWR012")
 					(unit 1)
 				)
 				(path "/16213bc9-ed22-4e8b-8e21-f5cd88729472/a83cc724-240f-4e24-86d0-fe129e515c9d"
-					(reference "#PWR013")
+					(reference "#PWR015")
 					(unit 1)
 				)
 				(path "/16213bc9-ed22-4e8b-8e21-f5cd88729472/f65a2aaa-bdb9-4087-a40a-8b8d146426dc"
-					(reference "#PWR016")
+					(reference "#PWR018")
 					(unit 1)
 				)
 				(path "/16213bc9-ed22-4e8b-8e21-f5cd88729472/9b53e793-8acb-49d6-9671-6c75b365109f"
-					(reference "#PWR019")
+					(reference "#PWR021")
 					(unit 1)
 				)
@@
 			)
 		)
-		(property "Footprint" "Resistor_SMD:R_0805_2012Metric_Pad1.20x1.40mm_HandSolder"
+		(property "Footprint" "Resistor_SMD:R_0603_1608Metric_Pad0.98x0.95mm_HandSolder"
 			(at 159.512 110.49 90)
 			(effects
@@
 			)
 		)
-		(property "Footprint" "Resistor_SMD:R_0805_2012Metric_Pad1.20x1.40mm_HandSolder"
+		(property "Footprint" "Resistor_SMD:R_0603_1608Metric_Pad0.98x0.95mm_HandSolder"
 			(at 168.91 93.472 90)
 			(effects
@@
 				(path "/16213bc9-ed22-4e8b-8e21-f5cd88729472/9b53e793-8acb-49d6-9671-6c75b365109f"
 					(reference "R17")
-					(unit 1)
-				)
-			)
-		)
-	)
-	(symbol
-		(lib_id "Connector:TestPoint")
-		(at 203.2 95.25 0)
-		(unit 1)
-		(exclude_from_sim no)
-		(in_bom yes)
-		(on_board yes)
-		(dnp no)
-		(property "Reference" "TP2"
-			(at 204.978 91.948 0)
-			(effects
-				(font
-					(size 1.27 1.27)
-				)
-				(justify left)
-			)
-		)
-		(property "Value" "TestPoint"
-			(at 205.74 93.2179 0)
-			(effects
-				(font
-					(size 1.27 1.27)
-				)
-				(justify left)
-				(hide yes)
-			)
-		)
-		(property "Footprint" ""
-			(at 208.28 95.25 0)
-			(effects
-				(font
-					(size 1.27 1.27)
-				)
-				(hide yes)
-			)
-		)
-		(property "Datasheet" "~"
-			(at 208.28 95.25 0)
-			(effects
-				(font
-					(size 1.27 1.27)
-				)
-				(hide yes)
-			)
-		)
-		(property "Description" "test point"
-			(at 203.2 95.25 0)
-			(effects
-				(font
-					(size 1.27 1.27)
-				)
-				(hide yes)
-			)
-		)
-		(pin "1"
-		)
-		(instances
-			(project "Kicad"
-				(path "/16213bc9-ed22-4e8b-8e21-f5cd88729472/72d653c3-8f6f-4150-b7cd-d5c98c703715"
-					(reference "TP2")
-					(unit 1)
-				)
-				(path "/16213bc9-ed22-4e8b-8e21-f5cd88729472/a83cc724-240f-4e24-86d0-fe129e515c9d"
-					(reference "TP3")
-					(unit 1)
-				)
-				(path "/16213bc9-ed22-4e8b-8e21-f5cd88729472/f65a2aaa-bdb9-4087-a40a-8b8d146426dc"
-					(reference "TP4")
-					(unit 1)
-				)
-				(path "/16213bc9-ed22-4e8b-8e21-f5cd88729472/9b53e793-8acb-49d6-9671-6c75b365109f"
-					(reference "TP5")
 					(unit 1)
 				)
@@
 				)
 				(path "/16213bc9-ed22-4e8b-8e21-f5cd88729472/f65a2aaa-bdb9-4087-a40a-8b8d146426dc"
+					(reference "U8")
+					(unit 2)
+				)
+				(path "/16213bc9-ed22-4e8b-8e21-f5cd88729472/9b53e793-8acb-49d6-9671-6c75b365109f"
 					(reference "U9")
-					(unit 2)
-				)
-				(path "/16213bc9-ed22-4e8b-8e21-f5cd88729472/9b53e793-8acb-49d6-9671-6c75b365109f"
-					(reference "U10")
 					(unit 2)
 				)
@@
 			)
 		)
-		(property "Footprint" "Resistor_SMD:R_0805_2012Metric_Pad1.20x1.40mm_HandSolder"
+		(property "Footprint" "Resistor_SMD:R_0603_1608Metric_Pad0.98x0.95mm_HandSolder"
 			(at 172.212 87.63 90)
 			(effects
@@
 		(on_board yes)
 		(dnp no)
-		(property "Reference" "#PWR09"
+		(property "Reference" "#PWR011"
 			(at 173.99 85.09 0)
 			(effects
@@
 			(project "Kicad"
 				(path "/16213bc9-ed22-4e8b-8e21-f5cd88729472/72d653c3-8f6f-4150-b7cd-d5c98c703715"
-					(reference "#PWR09")
+					(reference "#PWR011")
 					(unit 1)
 				)
 				(path "/16213bc9-ed22-4e8b-8e21-f5cd88729472/a83cc724-240f-4e24-86d0-fe129e515c9d"
-					(reference "#PWR012")
+					(reference "#PWR014")
 					(unit 1)
 				)
 				(path "/16213bc9-ed22-4e8b-8e21-f5cd88729472/f65a2aaa-bdb9-4087-a40a-8b8d146426dc"
-					(reference "#PWR015")
+					(reference "#PWR017")
 					(unit 1)
 				)
 				(path "/16213bc9-ed22-4e8b-8e21-f5cd88729472/9b53e793-8acb-49d6-9671-6c75b365109f"
-					(reference "#PWR018")
+					(reference "#PWR020")
 					(unit 1)
 				)
@@
 			)
 		)
-		(property "Footprint" "Resistor_SMD:R_0805_2012Metric_Pad1.20x1.40mm_HandSolder"
+		(property "Footprint" "Resistor_SMD:R_0603_1608Metric_Pad0.98x0.95mm_HandSolder"
 			(at 159.512 100.33 90)
 			(effects
@@
 					(unit 1)
 				)
+			)
+		)
+	)
+	(symbol
+		(lib_id "Jumper:SolderJumper_2_Open")
+		(at 204.47 97.79 0)
+		(unit 1)
+		(exclude_from_sim no)
+		(in_bom yes)
+		(on_board yes)
+		(dnp no)
+		(property "Reference" "JP5"
+			(at 203.962 94.234 0)
+			(effects
+				(font
+					(size 1.27 1.27)
+				)
+			)
+		)
+		(property "Value" "SolderJumper_2_Open"
+			(at 204.47 93.98 0)
+			(effects
+				(font
+					(size 1.27 1.27)
+				)
+				(hide yes)
+			)
+		)
+		(property "Footprint" "Jumper:SolderJumper-2_P1.3mm_Open_TrianglePad1.0x1.5mm"
+			(at 204.47 97.79 0)
+			(effects
+				(font
+					(size 1.27 1.27)
+				)
+				(hide yes)
+			)
+		)
+		(property "Datasheet" "~"
+			(at 204.47 97.79 0)
+			(effects
+				(font
+					(size 1.27 1.27)
+				)
+				(hide yes)
+			)
+		)
+		(property "Description" "Solder Jumper, 2-pole, open"
+			(at 204.47 97.79 0)
+			(effects
+				(font
+					(size 1.27 1.27)
+				)
+				(hide yes)
+			)
+		)
+		(pin "1"
+		)
+		(pin "2"
+		)
+		(instances
+			(project "Kicad"
+				(path "/16213bc9-ed22-4e8b-8e21-f5cd88729472/72d653c3-8f6f-4150-b7cd-d5c98c703715"
+					(reference "JP5")
+					(unit 1)
+				)
+				(path "/16213bc9-ed22-4e8b-8e21-f5cd88729472/a83cc724-240f-4e24-86d0-fe129e515c9d"
+					(reference "JP6")
+					(unit 1)
+				)
+				(path "/16213bc9-ed22-4e8b-8e21-f5cd88729472/f65a2aaa-bdb9-4087-a40a-8b8d146426dc"
+					(reference "JP7")
+					(unit 1)
+				)
+				(path "/16213bc9-ed22-4e8b-8e21-f5cd88729472/9b53e793-8acb-49d6-9671-6c75b365109f"
+					(reference "JP8")
+					(unit 1)
+				)

Commit message: modif
Parts:
- added unit 3 of U3
Connections:
- new net +15V: U3.8 (V+)
- new net -15V: U3.4 (V-)
Changed lines of the file:
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@@
+	(wire
+		(pts
+			(xy 218.44 49.53) (xy 218.44 50.8)
+		)
+		(stroke
+			(width 0)
+			(type default)
+		)
+	)
 	(wire
 		(pts
@@
 	(wire
 		(pts
+			(xy 226.06 49.53) (xy 218.44 49.53)
+		)
+		(stroke
+			(width 0)
+			(type default)
+		)
+	)
+	(wire
+		(pts
 			(xy 161.29 95.25) (xy 161.29 96.52)
 		)
@@
 	(wire
 		(pts
+			(xy 218.44 67.31) (xy 218.44 66.04)
+		)
+		(stroke
+			(width 0)
+			(type default)
+		)
+	)
+	(wire
+		(pts
 			(xy 173.99 81.28) (xy 173.99 83.82)
 		)
@@
 	(wire
 		(pts
+			(xy 218.44 67.31) (xy 227.33 67.31)
+		)
+		(stroke
+			(width 0)
+			(type default)
+		)
+	)
+	(wire
+		(pts
 			(xy 193.04 97.79) (xy 190.5 97.79)
 		)
@@
 			(width 0)
 			(type default)
+		)
+	)
+	(global_label "+15V"
+		(shape input)
+		(at 226.06 49.53 0)
+		(fields_autoplaced yes)
+		(effects
+			(font
+				(size 1.27 1.27)
+			)
+			(justify left)
+		)
+		(property "Intersheetrefs" "${INTERSHEET_REFS}"
+			(at 234.1252 49.53 0)
+			(effects
+				(font
+					(size 1.27 1.27)
+				)
+				(justify left)
+				(hide yes)
+			)
+		)
+	)
+	(global_label "-15V"
+		(shape input)
+		(at 227.33 67.31 0)
+		(fields_autoplaced yes)
+		(effects
+			(font
+				(size 1.27 1.27)
+			)
+			(justify left)
+		)
+		(property "Intersheetrefs" "${INTERSHEET_REFS}"
+			(at 235.3952 67.31 0)
+			(effects
+				(font
+					(size 1.27 1.27)
+				)
+				(justify left)
+				(hide yes)
+			)
 		)
 	)
@@
 			)
 			(justify left)
+		)
+	)
+	(symbol
+		(lib_id "Amplifier_Operational:OP275")
+		(at 220.98 58.42 0)
+		(unit 3)
+		(exclude_from_sim no)
+		(in_bom yes)
+		(on_board yes)
+		(dnp no)
+		(property "Reference" "U3"
+			(at 220.218 56.896 0)
+			(effects
+				(font
+					(size 1.27 1.27)
+				)
+				(justify left)
+			)
+		)
+		(property "Value" "OP275"
+			(at 220.218 59.436 0)
+			(effects
+				(font
+					(size 1.27 1.27)
+				)
+				(justify left)
+			)
+		)
+		(property "Footprint" "Package_SO:SOIC-8_3.9x4.9mm_P1.27mm"
+			(at 220.98 58.42 0)
+			(effects
+				(font
+					(size 1.27 1.27)
+				)
+				(hide yes)
+			)
+		)
+		(property "Datasheet" "https://www.analog.com/media/en/technical-documentation/data-sheets/OP275.pdf"
+			(at 220.98 58.42 0)
+			(effects
+				(font
+					(size 1.27 1.27)
+				)
+				(hide yes)
+			)
+		)
+		(property "Description" "Dual Bipolar/JFET, Audio Operational Amplifier, DIP-8/SOIC-8"
+			(at 220.98 58.42 0)
+			(effects
+				(font
+					(size 1.27 1.27)
+				)
+				(hide yes)
+			)
+		)
+		(pin "3"
+		)
+		(pin "7"
+		)
+		(pin "2"
+		)
+		(pin "6"
+		)
+		(pin "4"
+		)
+		(pin "8"
+		)
+		(pin "5"
+		)
+		(pin "1"
+		)
+		(instances
+			(project "Kicad"
+				(path "/16213bc9-ed22-4e8b-8e21-f5cd88729472/72d653c3-8f6f-4150-b7cd-d5c98c703715"
+					(reference "U3")
+					(unit 3)
+				)
+				(path "/16213bc9-ed22-4e8b-8e21-f5cd88729472/a83cc724-240f-4e24-86d0-fe129e515c9d"
+					(reference "U4")
+					(unit 3)
+				)
+				(path "/16213bc9-ed22-4e8b-8e21-f5cd88729472/f65a2aaa-bdb9-4087-a40a-8b8d146426dc"
+					(reference "U5")
+					(unit 3)
+				)
+				(path "/16213bc9-ed22-4e8b-8e21-f5cd88729472/9b53e793-8acb-49d6-9671-6c75b365109f"
+					(reference "U6")
+					(unit 3)
+				)
+			)
 		)
 	)
@@
 				)
 				(path "/16213bc9-ed22-4e8b-8e21-f5cd88729472/f65a2aaa-bdb9-4087-a40a-8b8d146426dc"
-					(reference "U8")
+					(reference "U5")
 					(unit 1)
 				)
 				(path "/16213bc9-ed22-4e8b-8e21-f5cd88729472/9b53e793-8acb-49d6-9671-6c75b365109f"
-					(reference "U9")
+					(reference "U6")
 					(unit 1)
 				)
@@
 		)
 		(property "Footprint" "Library.pretty_Conn_Coax1:Conn_CoaxE"
-			(at 134.62 92.71 0)
+			(at 135.382 85.344 0)
 			(effects
 				(font
@@
 		)
 		(property "Description" "coaxial connector (BNC, SMA, SMB, SMC, Cinch/RCA, LEMO, ...)"
-			(at 134.62 92.71 0)
+			(at 133.604 100.584 0)
 			(effects
 				(font
@@
 				(path "/16213bc9-ed22-4e8b-8e21-f5cd88729472/9b53e793-8acb-49d6-9671-6c75b365109f"
 					(reference "J4")
+					(unit 1)
+				)
+				(path "/16213bc9-ed22-4e8b-8e21-f5cd88729472"
+					(reference "J1")
 					(unit 1)
 				)
@@
 				)
 				(path "/16213bc9-ed22-4e8b-8e21-f5cd88729472/f65a2aaa-bdb9-4087-a40a-8b8d146426dc"
-					(reference "U8")
+					(reference "U5")
 					(unit 2)
 				)
 				(path "/16213bc9-ed22-4e8b-8e21-f5cd88729472/9b53e793-8acb-49d6-9671-6c75b365109f"
-					(reference "U9")
+					(reference "U6")
 					(unit 2)
 				)

Commit message: modif
Parts:
- renumbered J1 to JC1
Changed lines of the file:
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@@
 		(on_board yes)
 		(dnp no)
-		(property "Reference" "J1"
+		(property "Reference" "JC1"
 			(at 135.636 98.298 0)
 			(effects
@@
 			(project "Kicad"
 				(path "/16213bc9-ed22-4e8b-8e21-f5cd88729472/72d653c3-8f6f-4150-b7cd-d5c98c703715"
-					(reference "J1")
+					(reference "JC1")
 					(unit 1)
 				)
 				(path "/16213bc9-ed22-4e8b-8e21-f5cd88729472/a83cc724-240f-4e24-86d0-fe129e515c9d"
-					(reference "J2")
+					(reference "JC2")
 					(unit 1)
 				)
 				(path "/16213bc9-ed22-4e8b-8e21-f5cd88729472/f65a2aaa-bdb9-4087-a40a-8b8d146426dc"
-					(reference "J3")
+					(reference "JC3")
 					(unit 1)
 				)
 				(path "/16213bc9-ed22-4e8b-8e21-f5cd88729472/9b53e793-8acb-49d6-9671-6c75b365109f"
-					(reference "J4")
+					(reference "JC4")
 					(unit 1)
 				)
-				(path "/16213bc9-ed22-4e8b-8e21-f5cd88729472"
-					(reference "J1")
-					(unit 1)
-				)

Commit message: modif
Parts:
- R6: value 8.25k -> 4.5k
Changed lines of the file:
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@@
 			)
 		)
-		(property "Value" "8.25k"
+		(property "Value" "4.5k"
 			(at 163.83 101.5999 0)
 			(effects
