File: Hardware/Kicad_Carte_Acquisition/Kicad.kicad_pcb (KiCad board)
At the start: 2 copper layers, 208.2 x 123 mm, 97 parts, among them P1 DA15_Receptacle_MountingHoles, U1 TMP-15-215, U10 LV25-P, U11 OP275, U12 LV25-P, U2 LM2937xS, U3 OP275, U4 OP275, U5 OP275, U6 OP275, U7 OP275, U8 LV25-P, U9 OP275

Commit message: modif
Parts:
- moved D3 21.2 mm to (244.4, 138.1)
- moved R3 21.2 mm to (239.7, 138.1)
- moved JC3 14.0 mm to (134.0, 36.6), turned to 90 degrees
- moved JC4 14.0 mm to (120.0, 36.6), turned to 90 degrees
- moved JP13 10.1 mm to (155.3, 109.6)
- moved JP11 9.19 mm to (186.0, 109.6)
- moved JP8 8.78 mm to (136.0, 73.9)
- moved JP9 8.69 mm to (216.0, 109.6)
- moved JP4 2.12 mm to (224.5, 130.1), turned to 180 degrees
- moved R24 1.00 mm to (228.0, 103.1)
- moved C13 0.71 mm to (221.5, 107.1)
- moved C14 0.71 mm to (191.5, 107.1)
- moved C9 0.64 mm to (158.1, 45.6)
- moved C1 0.50 mm to (232.5, 125.1)
- moved C10 0.50 mm to (144.0, 45.6)
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Connections:
- U10 pad 6: +15V -> -15V
- U12 pad 6: +15V -> -15V
- U8 pad 6: +15V -> -15V
Routing:
- net -15V: track 0.00 -> 254.5 mm, vias 0 -> 4
- net +15V: track 0.00 -> 254.4 mm, vias 0 -> 2
- net GND: track 0.00 -> 238.4 mm
- net +3V3: track 0.00 -> 136.6 mm
- net Neutre: track 0.00 -> 95.6 mm
- net Net-(U12-HV+): track 0.00 -> 34.0 mm
- net Net-(JC3-In): track 0.00 -> 25.7 mm
- net Net-(JC4-In): track 0.00 -> 25.7 mm
- net Net-(JC2-In): track 0.00 -> 25.3 mm
- net Net-(JC1-In): track 0.00 -> 24.7 mm
- net Net-(JB6-Pin_1): track 0.00 -> 21.7 mm
- net Net-(U10-HV+): track 0.00 -> 19.5 mm
- net Net-(JP4-B): track 0.00 -> 18.6 mm
- net Net-(U11B-+): track 0.00 -> 17.0 mm
- net Net-(U9B-+): track 0.00 -> 16.9 mm
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Other:
- board size 208.2 x 123 mm -> 208 x 123 mm

Commit message: modif
Parts:
- moved JP10 49.5 mm to (178.0, 121.1)
- moved JP12 25.4 mm to (172.0, 121.1)
- moved JP14 4.68 mm to (166.0, 121.1)
- moved R2 0.09 mm to (112.5, 139.1)
- turned D1 to 180 degrees
- turned R1 to 180 degrees
- turned R33 to 0 degrees
Routing:
- net GND: track 238.4 -> 835.2 mm, vias 0 -> 7
- net Vcurrent_ph2: track 0.00 -> 154.2 mm, vias 0 -> 1
- net Vcurrent_ph3: track 0.00 -> 135.1 mm, vias 0 -> 1
- net +15V: track 254.4 -> 386.9 mm, vias 2 -> 7
- net Vcurrent_ph1: track 0.00 -> 106.7 mm, vias 0 -> 1
- net Vcurrent_neutre: track 0.00 -> 75.8 mm, vias 0 -> 1
- net +3V3: track 136.6 -> 209.8 mm, vias 0 -> 2
- net Net-(JP1-A): track 0.00 -> 68.6 mm
- net Net-(JP10-A): track 0.00 -> 53.9 mm, vias 0 -> 2
- net Net-(JP3-A): track 0.00 -> 42.7 mm
- net Net-(JP2-A): track 0.00 -> 41.6 mm
- net Net-(JP8-A): track 0.00 -> 35.0 mm, vias 0 -> 2
- net Net-(JP12-A): track 0.00 -> 31.3 mm, vias 0 -> 2
- net -15V: track 254.5 -> 284.8 mm, vias 4 -> 7
- net Vph1: track 0.00 -> 26.6 mm
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
Commit message: modif
Parts:
- moved JC4 20.0 mm to (100.0, 36.6)
- moved F1 15.3 mm to (66.0, 70.1)
- moved JB5 15.0 mm to (65.5, 43.6)
- moved JB6 15.0 mm to (83.5, 43.6)
- moved JC3 14.0 mm to (120.0, 36.6)
- moved JC2 8.00 mm to (140.0, 36.6)
- moved JC1 2.00 mm to (160.0, 36.6)
Routing:
- net GND: track 835.2 -> 869.8 mm
- net Net-(U1-AC(L)): track 14.8 -> 31.8 mm
- net Net-(JB6-Pin_1): track 21.7 -> 34.7 mm
- net Net-(JC2-In): track 25.3 -> 19.3 mm
- net Net-(R10-Pad1): track 10.8 -> 15.8 mm
- net Net-(JC4-In): track 25.7 -> 30.5 mm, vias 0 -> 1
- net Net-(JB5-Pin_1): track 13.0 -> 15.4 mm
- net Net-(JC3-In): track 25.7 -> 23.6 mm
- net Net-(JC1-In): track 24.7 -> 24.5 mm, vias 0 -> 1

Commit message: maj
Routing:
- net GND: track 869.8 -> 44.9 mm, vias 7 -> 10
- net Vcurrent_ph2: track 154.2 -> 166.5 mm
- net +15V: track 386.9 -> 375.1 mm
- net Vcurrent_ph1: track 106.7 -> 113.0 mm
- net Vcurrent_ph3: track 135.1 -> 140.5 mm
- net Net-(R10-Pad1): track 15.8 -> 10.8 mm
- net -15V: track 284.8 -> 286.6 mm, vias 7 -> 5
Other:
- board text added: "+15V"
- board text added: "-15V"
- board text added: "230V/Neutre"
- board text added: "230V/Phase"
- board text added: "GND"
- board text added: "Neutre"
- board text added: "Phase 1"
- board text added: "Phase 2"
- board text added: "Phase 3"
- board text added: "Vcurrent 1"
- board text added: "Vcurrent 2"
- board text added: "Vcurrent 3"
- board text added: "Vcurrent neutre"

Commit message: modif
Parts:
- moved R13 1.12 mm to (130.0, 51.6), turned to 180 degrees
- moved R17 1.12 mm to (116.0, 51.6), turned to 180 degrees
- moved R9 1.12 mm to (144.0, 51.6), turned to 180 degrees
- moved R5 0.77 mm to (158.0, 51.1), turned to 180 degrees
- moved C4 0.50 mm to (153.0, 51.1)
- moved C5 0.50 mm to (139.0, 51.1)
- moved C6 0.50 mm to (125.0, 51.1)
Routing:
- net Net-(R10-Pad1): track 10.8 -> 2.84 mm
- net Net-(R13-Pad2): track 10.9 -> 15.0 mm
- net Net-(R17-Pad2): track 11.2 -> 14.8 mm
- net +15V: track 375.1 -> 378.3 mm
- net Net-(R5-Pad2): track 11.1 -> 14.0 mm
- net +3V3: track 210.3 -> 213.2 mm
- net Net-(JP8-A): track 35.0 -> 35.6 mm
- net Net-(U3B-+): track 4.89 -> 4.34 mm
- net GND: vias 10 -> 11
Other:
- board text added: "Ingénieurs projets: Hicham IDIR Julien SAINT-LEGER Jingwen ZHANG Anas KHOUFAIFY"
- board text added: "Projet Analyseur de réseau électrique - Carte d'acqusition -"

Commit message: modif
Parts:
- R10, R14, R18, R6: value 8.25k -> 4.5k
- moved P1 9.29 mm to (155.4, 152.6)
Routing:
- net GND: track 44.9 -> 2.01 mm, vias 11 -> 6
- net Net-(JP1-A): track 68.6 -> 79.8 mm
- net Net-(JP2-A): track 41.6 -> 50.7 mm
- net +15V: track 378.3 -> 386.7 mm
- net Net-(JP3-A): track 42.7 -> 49.7 mm
- net Vph1: track 26.6 -> 32.8 mm
- net Vph2: track 25.2 -> 29.0 mm
- net Net-(U12-HV+): track 34.0 -> 37.5 mm
- net Vph3: track 23.9 -> 26.5 mm
- net Vcurrent_ph2: track 166.5 -> 168.9 mm
- net Vcurrent_ph3: track 140.5 -> 142.3 mm
- net Net-(U11B-+): track 17.0 -> 17.7 mm
- net Vcurrent_ph1: track 113.0 -> 113.5 mm

Commit message: modif
Parts:
- removed P1: DA15_Receptacle_MountingHoles, Library.pretty_Dsub_15_Female:Dsub_15_Female_E
- added J1: DA15_Receptacle, Library.pretty_SUBD_F:618015231321, F.Cu at (165.2, 140.9)
Routing:
- net GND: track 2.01 -> 0.00 mm
- net +15V: track 386.7 -> 387.2 mm
- net Vph1: track 32.8 -> 32.3 mm
