File: Hardware/Kicad_Carte_Traitement/Kicad.kicad_sch (KiCad schematic)
At the start: 51 parts, among them J1 Conn_01x01, J2 Conn_01x01, J3 Conn_01x01, J4 Conn_01x01, J5 DA15_Receptacle_MountingHoles, U1 LV25-P, U10 OP275, U11 OP275, U12 OP275, U13 OP275, U14 OP275, U15 OP275, U2 LV25-P, U3 LV25-P, U4 OP275, U5 OP275, U6 OP275, U7 LM2937xS, U8 OP275, U9 OP275

Commit message: MAJ
Parts:
- removed J1, J2, J3, J4: Conn_01x01, Connector:Banana_Cliff_FCR7350B_S16N-PC_Horizontal, symbol Connector_Generic:Conn_01x01
- removed R1, R10, R11, R12, R13, R14, R15, R16, R17, R18, R19, R2, R20, R21, R22, R23, R24, R25, R26, R27, R28, R29, R3, R30, R31, R4, R5, R6, R7, R8, R9: R, symbol Device:R
- removed U1, U2, U3: LV25-P, Sensor_Voltage:LEM_LV25-P, symbol Sensor_Voltage:LV25-P
- removed U10, U11, U12, U13, U14, U15, U4, U5, U6, U8, U9: OP275, symbol Amplifier_Operational:OP275
- removed U7: LM2937xS, Package_TO_SOT_SMD:TO-263-3_TabPin2, symbol Regulator_Linear:LM2937xS
- added U2: STM32G474RETx, Package_QFP:LQFP-64_10x10mm_P0.5mm, symbol MCU_ST_STM32G4:STM32G474RETx
- added WE1: ~, Library:test, symbol New_Library:test
Connections:
- new net: U2.15 (VSS), U2.31 (VSS), U2.47 (VSS), U2.63 (VSS)

Commit message: MAJ
Parts:
- added C1: 4u7, symbol Device:C
- added C2, C3, C7, C8: 100n, symbol Device:C
- added C4: 10n, symbol Device:C
- added C5, C6: 1u, symbol Device:C
- added D1: LED Orange 1,8v 3,5mA, symbol Device:LED
- added D2: LED Green 2,8v 2mA, symbol Device:LED
- added H1, H2, H3, H4: MountingHole_Pad, symbol Mechanical:MountingHole_Pad
- added J1: Conn_02x07_Odd_Even, symbol Connector_Generic:Conn_02x07_Odd_Even
- added L1: 39n, symbol Device:L
- added OLED1306: ~, Library:OLED, symbol OLED:SSD1306
- added R1: 180, symbol Device:R
- added R2: 240, symbol Device:R
- added R3: 10k, symbol Device:R
- added S1: ~, Switch:Tact_switch, symbol switch:Tact_switch
Connections:
- net USART2_TX: now reaches U2.14 (PA2)
- net USART2_TX: now also J1.14 (Pin_14)
- net GND: now reaches U2.15 (VSS), U2.31 (VSS), U2.47 (VSS), U2.63 (VSS)
- net GND: now also J5.0 (PAD), J5.8, U2.27 (VSSA), WE1.2 (GND), C1.2, C2.2, C3.2, C4.2, C5.2, C6.2, C7.2, C8.2, H1.1, H2.1, H3.1, H4.1, J1.11 (Pin_11), J1.5 (Pin_5), J1.7 (Pin_7), OLED1306. (VCC), R1.2, R2.2, S1.3, S1.4
- net +3.3V: now reaches U2.16 (VDD)
- net +3.3V: now also U2.32 (VDD), U2.48 (VDD), U2.64 (VDD), WE1.3 (OUT), C1.1, C2.1, C3.1, D2.2 (A), J1.3 (Pin_3), L1.2, OLED1306. (VCC), R3.1
- net USART2_RX: now reaches U2.17 (PA3)
- net USART2_RX: now also J1.13 (Pin_13)
- net LED_STATUS: now reaches U2.18 (PA4)
- net LED_STATUS: now also D1.2 (A)
- net at U2.28 (VREF+): now also C6.1, C7.1
- net +3.3VA: now reaches U2.29 (VDDA)
- net +3.3VA: now also C4.1, C5.1, L1.1
- net SWDIO: now reaches U2.49 (PA13)
- net SWDIO: now also J1.4 (Pin_4)
- net SWCLK: now reaches U2.50 (PA14)
- net SWCLK: now also J1.6 (Pin_6)
- net I2C-SDA: now reaches U2.60 (PB7)
- net I2C-SDA: now also OLED1306. (VCC)
- net I2C-SCL: now reaches U2.61 (PB8)
- net I2C-SCL: now also OLED1306. (VCC)
- net NRST: now reaches U2.7 (PG10)
- net NRST: now also J1.12 (Pin_12)
- net Vph1: now reaches J5.1
- net Vcurrent_ph2: now reaches J5.10 (P10)
- net Vcurrent_ph3: now reaches J5.11 (P111)
- net +15V: now reaches J5.15 (P15)
- net +15V: now also WE1.1 (In)
- net Vph2: now reaches J5.2
- net Vph3: now reaches J5.3
- net Vcurrent_neutre: now reaches J5.4
- net Vcurrent_ph1: now reaches J5.9 (P9)
- new net: C8.1, R3.2, S1.1, S1.2
- new net: D1.1 (K), R1.1
- new net: D2.1 (K), R2.1
- no-connect marks 0 -> 5
Other:
- note added: "Mounting Holes"
- note added: "OLED"
- note added: "Power Supply"
- note added: "STM32 Microcontroller"
- note added: "SWD Connector"
- moved on the sheet: U2, WE1

Commit message: MAJ
Parts:
- added C10, C11, C9: 100n, symbol Device:C
- added R4, R5, R6: 10k, symbol Device:R
- added S2, S3, S4: ~, Switch:Tact_switch, symbol switch:Tact_switch
- J5: footprint (none) -> Library.pretty_SUBD:SUB_D
Connections:
- net +15V: now also J5.9 (P9); no longer J5.15 (P15)
- net +3.3V: now also R4.1, R5.1, R6.1
- net GND: now also J5.1, C10.2, C11.2, C9.2, S2.3, S2.4, S3.3, S3.4, S4.3, S4.4; no longer J5.8
- net I2C-SCL: now also C9.1, R4.2, S2.1, S2.2
- net I2C-SDA: now also C10.1, C11.1, R5.2, R6.2, S3.1, S3.2, S4.1, S4.2
- net NRST: now also C8.1, R3.2, S1.1, S1.2
- net Vcurrent_neutre: now also J5.5, U2.42 (PA8); no longer J5.4
- net Vcurrent_ph1: now also J5.15 (P15), U2.37 (PB15); no longer J5.9 (P9)
- net Vcurrent_ph2: now also J5.14 (P14), U2.25 (PB1); no longer J5.10 (P10)
- net Vcurrent_ph3: now also J5.13 (P13), U2.36 (PB14); no longer J5.11 (P111)
- net Vph1: now also J5.8, U2.5 (PF0); no longer J5.1
- net Vph2: now also J5.7, U2.6 (PF1); no longer J5.2
- net Vph3: now also J5.6, U2.24 (PB0); no longer J5.3
- no-connect marks 5 -> 11
Other:
- note added: "Button"
- note added: "Menu +"
- note added: "Menu -"
- note added: "RESET"
- note added: "START"
- note added: "SUB_D Connector"
- moved on the sheet: C1, C2, C3, C4, C5, C6, C7, C8, D1, D2, H1, H2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

Commit message: MAJ
Parts:
- added J2: POWER, symbol Connector_Generic:Conn_01x02
- added J6: INPUT, symbol Connector_Generic:Conn_02x04_Counter_Clockwise
Connections:
- net +15V: now also J2.1 (Pin_1)
- net GND: now also S1.2, S2.2, S3.2, S4.2, J2.2 (Pin_2), J6.5 (Pin_5); no longer S1.3, S2.3, S3.3, S4.3
- net I2C-SCL: now also S2.3; no longer S2.2
- net I2C-SDA: now also S3.3, S4.3; no longer S3.2, S4.2
- net NRST: now also S1.3; no longer S1.2
- net Vcurrent_neutre: now also J6.6 (Pin_6)
- net Vcurrent_ph1: now also J6.2 (Pin_2)
- net Vcurrent_ph2: now also J6.4 (Pin_4)
- net Vcurrent_ph3: now also J6.7 (Pin_7)
- net Vph1: now also J6.1 (Pin_1)
- net Vph2: now also J6.3 (Pin_3)
- net Vph3: now also J6.8 (Pin_8)
- no-connect marks 11 -> 49
Other:
- note added: "IO Connectors"
- moved on the sheet: S1, S2, S3, S4

Commit message: MAJ
Parts:
- removed J2: POWER, symbol Connector_Generic:Conn_01x02
- removed J5: DA15_Receptacle_MountingHoles, Library.pretty_SUBD:SUB_D, symbol Connector:DA15_Receptacle_MountingHoles
- removed J6: INPUT, symbol Connector_Generic:Conn_02x04_Counter_Clockwise
- removed OLED1306: ~, Library:OLED, symbol OLED:SSD1306
- added J2: DA15_Receptacle, Library.pretty_SUBD_F:618015231321, symbol Connector:DA15_Receptacle
- added OLED1: ~, Library:OLED, symbol OLED:SSD1306
- added R10, R7, R8, R9: 10k, Resistor_SMD:R_0603_1608Metric_Pad0.98x0.95mm_HandSolder, symbol Device:R
- added TP1: START, Connector_Pin:Pin_D1.2mm_L10.2mm_W2.9mm_FlatFork, symbol Connector:TestPoint
- added TP10: Vcurrent_ph1, Connector_Pin:Pin_D1.2mm_L10.2mm_W2.9mm_FlatFork, symbol Connector:TestPoint
- added TP11: I2C-SDA, Connector_Pin:Pin_D1.2mm_L10.2mm_W2.9mm_FlatFork, symbol Connector:TestPoint
- added TP12: I2C-SCL, Connector_Pin:Pin_D1.2mm_L10.2mm_W2.9mm_FlatFork, symbol Connector:TestPoint
- added TP13: RESET, Connector_Pin:Pin_D1.2mm_L10.2mm_W2.9mm_FlatFork, symbol Connector:TestPoint
- added TP2: Vph1, Connector_Pin:Pin_D1.2mm_L10.2mm_W2.9mm_FlatFork, symbol Connector:TestPoint
- added TP3: Vph2, Connector_Pin:Pin_D1.2mm_L10.2mm_W2.9mm_FlatFork, symbol Connector:TestPoint
- added TP4: Menu+, Connector_Pin:Pin_D1.2mm_L10.2mm_W2.9mm_FlatFork, symbol Connector:TestPoint
- added TP5: Menu-, Connector_Pin:Pin_D1.2mm_L10.2mm_W2.9mm_FlatFork, symbol Connector:TestPoint
- added TP6: N, Connector_Pin:Pin_D1.2mm_L10.2mm_W2.9mm_FlatFork, symbol Connector:TestPoint
- added TP7: Vph3, Connector_Pin:Pin_D1.2mm_L10.2mm_W2.9mm_FlatFork, symbol Connector:TestPoint
- added TP8: Vcurrent_ph2, Connector_Pin:Pin_D1.2mm_L10.2mm_W2.9mm_FlatFork, symbol Connector:TestPoint
- added TP9: Vcurrent_ph3, Connector_Pin:Pin_D1.2mm_L10.2mm_W2.9mm_FlatFork, symbol Connector:TestPoint
- C1, C2, C3, C4, C5, C6, C7: footprint (none) -> Capacitor_SMD:C_0603_1608Metric_Pad1.08x0.95mm_HandSolder
- C10, C11, C8, C9: value 100n -> 10n; footprint (none) -> Capacitor_SMD:C_0603_1608Metric_Pad1.08x0.95mm_HandSolder
- D1, D2: footprint (none) -> LED_SMD:LED_0603_1608Metric_Pad1.05x0.95mm_HandSolder
- H1, H2, H3, H4: footprint (none) -> MountingHole:MountingHole_3.2mm_M3_Pad
- J1: footprint (none) -> Connector_IDC:IDC-Header_2x07_P2.54mm_Vertical_SMD
- L1: footprint (none) -> Inductor_SMD:L_0603_1608Metric_Pad1.05x0.95mm_HandSolder
- R1, R2, R3, R4, R5, R6: footprint (none) -> Resistor_SMD:R_0603_1608Metric_Pad0.98x0.95mm_HandSolder
Connections:
- net +15V: now also J2.9 (P9)
- net GND: now also J2.1, OLED1.1 (GND)
- net I2C-SCL: now also OLED1.3 (SCL), TP12.1; no longer C9.1, R4.2, S2.1, S2.3
- net I2C-SDA: now also OLED1.4 (SDA), TP11.1; no longer C10.1, C11.1, R5.2, R6.2, S3.1, S3.3, S4.1, S4.3
- net NRST: now also R7.1, TP13.1; no longer C8.1
- net Vcurrent_neutre: now also J2.5, TP6.1
- net Vcurrent_ph1: now also J2.15 (P15), TP10.1
- net Vcurrent_ph2: now also J2.14 (P14), TP8.1
- net Vcurrent_ph3: now also J2.13 (P13), TP9.1
- net Vph1: now also J2.8, TP2.1
- net Vph2: now also J2.7, TP3.1
- net Vph3: now also J2.6, TP7.1
- net EXTI_MENU-: now reaches U2.2 (PC13)
- net EXTI_MENU-: now also R6.2, S4.1, S4.3, R10.1, TP5.1
- net EXTI_MENU+: now reaches U2.39 (PC7)
- net EXTI_MENU+: now also R5.2, S3.1, S3.3, R9.1, TP4.1
- net EXTI_START: now reaches U2.8 (PC0)
- net EXTI_START: now also R4.2, S2.1, S2.3, R8.1, TP1.1
- new net: C8.1, R7.2
- new net: C11.1, R10.2
- new net: C9.1, R8.2
- new net: C10.1, R9.2
- new net +3V3: OLED1.2 (VCC)
- no-connect marks 49 -> 46
Other:
- note removed: "IO Connectors"
- moved on the sheet: D2, R2, R3, R4, R5, R6, WE1

Commit message: maj ju
Parts:
- added TP14: +15v, Connector_Pin:Pin_D1.2mm_L10.2mm_W2.9mm_FlatFork, symbol Connector:TestPoint
Connections:
- net +15V: now also TP14.1
- net EXTI_MENU+: now also U2.33 (PB11); no longer U2.39 (PC7)
- net EXTI_MENU-: now also U2.34 (PB12); no longer U2.2 (PC13)
Other:
- moved on the sheet: TP4, TP5

Commit message: MAJ
Connections:
- net +3V3 is gone; now on net +3.3V: OLED1.2 (VCC)
Changed lines of the file:
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@@
+	)
+	(symbol
+		(lib_id "power:+3.3V")
+		(at 35.56 173.99 0)
+		(unit 1)
+		(exclude_from_sim no)
+		(in_bom yes)
+		(on_board yes)
+		(dnp no)
+		(fields_autoplaced yes)
+		(property "Reference" "#PWR011"
+			(at 35.56 177.8 0)
+			(effects
+				(font
+					(size 1.27 1.27)
+				)
+				(hide yes)
+			)
+		)
+		(property "Value" "+3.3V"
+			(at 35.56 168.91 0)
+			(effects
+				(font
+					(size 1.27 1.27)
+				)
+			)
+		)
+		(property "Footprint" ""
+			(at 35.56 173.99 0)
+			(effects
+				(font
+					(size 1.27 1.27)
+				)
+				(hide yes)
+			)
+		)
+		(property "Datasheet" ""
+			(at 35.56 173.99 0)
+			(effects
+				(font
+					(size 1.27 1.27)
+				)
+				(hide yes)
+			)
+		)
+		(property "Description" "Power symbol creates a global label with name \"+3.3V\""
+			(at 35.56 173.99 0)
+			(effects
+				(font
+					(size 1.27 1.27)
+				)
+				(hide yes)
+			)
+		)
+		(pin "1"
+		)
+		(instances
+			(project "Kicad"
+				(path "/16213bc9-ed22-4e8b-8e21-f5cd88729472"
+					(reference "#PWR011")
+					(unit 1)
+				)
+			)
+		)
 	)
 	(symbol
@@
 					(unit 1)
 				)
-			)
-		)
-	)
-	(symbol
-		(lib_id "power:+3V3")
-		(at 35.56 173.99 0)
-		(unit 1)
-		(exclude_from_sim no)
-		(in_bom yes)
-		(on_board yes)
-		(dnp no)
-		(fields_autoplaced yes)
-		(property "Reference" "#PWR011"
-			(at 35.56 177.8 0)
-			(effects
-				(font
-					(size 1.27 1.27)
-				)
-				(hide yes)
-			)
-		)
-		(property "Value" "+3V3"
-			(at 35.56 168.91 0)
-			(effects
-				(font
-					(size 1.27 1.27)
-				)
-			)
-		)
-		(property "Footprint" ""
-			(at 35.56 173.99 0)
-			(effects
-				(font
-					(size 1.27 1.27)
-				)
-				(hide yes)
-			)
-		)
-		(property "Datasheet" ""
-			(at 35.56 173.99 0)
-			(effects
-				(font
-					(size 1.27 1.27)
-				)
-				(hide yes)
-			)
-		)
-		(property "Description" "Power symbol creates a global label with name \"+3V3\""
-			(at 35.56 173.99 0)
-			(effects
-				(font
-					(size 1.27 1.27)
-				)
-				(hide yes)
-			)
-		)
-		(pin "1"
-		)
-		(instances
-			(project "Kicad"
-				(path "/16213bc9-ed22-4e8b-8e21-f5cd88729472"
-					(reference "#PWR011")
-					(unit 1)
-				)
